File: power_distribution_board/PDB.kicad_sch (KiCad schematic)
At the start: 0 parts

Commit message: Update Scheme & DEV_DOC
Parts:
- added CN1: XT60PW-M, easyeda2kicad:CONN-TH_XT60PW-M, symbol easyeda2kicad:XT60PW-M
- added R1: ASR-M-3-1F_C7370895, easyeda2kicad:RES-SMD_L6.3-W3.1-1, symbol easyeda2kicad:ASR-M-3-1F_C7370895
- added U1: INA226AIDGSR, easyeda2kicad:MSOP-10_L3.0-W3.0-P0.50-LS5.0-BL, symbol easyeda2kicad:INA226AIDGSR
- added U2: TPS54560DDAR, easyeda2kicad:SOIC-8_L5.0-W4.0-P1.27-LS6.0-BL-EP2.0, symbol easyeda2kicad:TPS54560DDAR

Commit message: Update Scheme
Parts:
- removed R1: ASR-M-3-1F_C7370895, easyeda2kicad:RES-SMD_L6.3-W3.1-1, symbol easyeda2kicad:ASR-M-3-1F_C7370895
- added C1, C2: CC0603KRX7R9BB104 (100nf , 0603 ,50v ,X7R), easyeda2kicad:C0603, symbol easyeda2kicad:CC0603KRX7R9BB104 (100nf , 0603 ,50v ,X7R)
- added C3: CL05A105KA5NQNC (1uf ,0402 ,25v,X5R), easyeda2kicad:C0402, symbol easyeda2kicad:CL05A105KA5NQNC (1uf ,0402 ,25v,X5R)
- added C4: CL21A226MAYNNNE (22uf , 0805 ,25v ,X5R), easyeda2kicad:C0805, symbol easyeda2kicad:CL21A226MAYNNNE (22uf , 0805 ,25v ,X5R)
- added R1: HOLR2725D-4W-0.5MR-1%, easyeda2kicad:R2725, symbol easyeda2kicad:HOLR2725D-4W-0.5MR-1%
- added R2, R3: FRC0603F4701TS (4.7kohm , 0603), easyeda2kicad:R0603, symbol easyeda2kicad:FRC0603F4701TS (4.7kohm , 0603)
- added R4, R5, R6: 603WAF0000T5E (0ohm , 0603), easyeda2kicad:R0603, symbol easyeda2kicad:0603WAF0000T5E (0ohm , 0603)
Connections:
- net 16.8V_BAT: now reaches CN1.2 (+)
- net 16.8V_BAT: now also R1.1, R5.2
- net GND: now reaches U2.7 (GND)
- net GND: now also U1.2 (A0), U1.7 (GND), C2.1, R6.2
- net at U1.1 (A1): now also R6.1
- net at U1.10 (VIN+): now also U1.8 (VBUS), C1.1, R5.1
- net SDA: now reaches U1.4 (SDA)
- net SDA: now also R3.1
- net SCL: now reaches U1.5 (SCL)
- net SCL: now also R2.1
- net 3V3: now reaches U1.6 (VS+)
- net 3V3: now also C2.2, R2.2, R3.2
- net at U1.9 (VIN-): now also C1.2, R4.1
- new net 16.8V: R1.2, R4.2
Other:
- note added: "Current Sensor I2C=0x40"
- note added: "PLACE CLOSE TO INA226 AS POSSIBLE"
- moved on the sheet: CN1, U1, U2

Commit message: Update Scheme
Parts:
- added R7: FRC0603F4701TS (4.7kohm , 0603), easyeda2kicad:R0603, symbol easyeda2kicad:FRC0603F4701TS (4.7kohm , 0603)
Connections:
- net 3V3: now also R7.2
- net ALERT: now reaches U1.3 (Alert)
- net ALERT: now also R7.1
Changed lines of the file:
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@@
+	)
+	(junction
+		(at 67.31 54.61)
+		(diameter 0)
+		(color 0 0 0 0)
 	)
 	(junction
@@
 	(wire
 		(pts
+			(xy 59.69 87.63) (xy 87.63 87.63)
+		)
+		(stroke
+			(width 0)
+			(type default)
+		)
+	)
+	(wire
+		(pts
 			(xy 129.54 59.69) (xy 129.54 72.39)
 		)
@@
 	(wire
 		(pts
+			(xy 59.69 54.61) (xy 67.31 54.61)
+		)
+		(stroke
+			(width 0)
+			(type default)
+		)
+	)
+	(wire
+		(pts
+			(xy 59.69 68.58) (xy 59.69 87.63)
+		)
+		(stroke
+			(width 0)
+			(type default)
+		)
+	)
+	(wire
+		(pts
 			(xy 135.89 85.09) (xy 135.89 82.55)
 		)
@@
 	(wire
 		(pts
+			(xy 96.52 77.47) (xy 87.63 77.47)
+		)
+		(stroke
+			(width 0)
+			(type default)
+		)
+	)
+	(wire
+		(pts
 			(xy 129.54 43.18) (xy 129.54 48.26)
 		)
@@
 	(wire
 		(pts
+			(xy 59.69 58.42) (xy 59.69 54.61)
+		)
+		(stroke
+			(width 0)
+			(type default)
+		)
+	)
+	(wire
+		(pts
 			(xy 67.31 68.58) (xy 67.31 82.55)
 		)
@@
 			(width 0)
 			(type default)
+		)
+	)
+	(wire
+		(pts
+			(xy 87.63 77.47) (xy 87.63 87.63)
+		)
+		(stroke
+			(width 0)
+			(type default)
+		)
+	)
+	(label "ALERT"
+		(at 76.2 87.63 0)
+		(effects
+			(font
+				(size 1.27 1.27)
+			)
+			(justify left bottom)
 		)
 	)
@@
 					(unit 1)
 				)
+			)
+		)
+	)
+	(symbol
+		(lib_id "easyeda2kicad:FRC0603F4701TS (4.7kohm , 0603)")
+		(at 59.69 63.5 90)
+		(unit 1)
+		(exclude_from_sim no)
+		(in_bom yes)
+		(on_board yes)
+		(dnp no)
+		(fields_autoplaced yes)
+		(property "Reference" "R7"
+			(at 57.404 63.5 0)
+			(do_not_autoplace yes)
+			(effects
+				(font
+					(size 1.27 1.27)
+				)
+			)
+		)
+		(property "Value" "FRC0603F4701TS (4.7kohm , 0603)"
+			(at 64.77 63.5 0)
+			(effects
+				(font
+					(size 1.27 1.27)
+				)
+				(hide yes)
+			)
+		)
+		(property "Footprint" "easyeda2kicad:R0603"
+			(at 67.31 63.5 0)
+			(effects
+				(font
+					(size 1.27 1.27)
+				)
+				(hide yes)
+			)
+		)
+		(property "Datasheet" ""
+			(at 59.69 63.5 0)
+			(effects
+				(font
+					(size 1.27 1.27)
+				)
+				(hide yes)
+			)
+		)
+		(property "Description" "4.7kΩ ±1% 100mW 0603 Thick Film Resistor"
+			(at 59.69 63.5 0)
+			(effects
+				(font
+					(size 1.27 1.27)
+				)
+				(hide yes)
+			)
+		)
+		(property "LCSC Part" "C2907034"
+			(at 69.85 63.5 0)
+			(effects
+				(font
+					(size 1.27 1.27)
+				)
+				(hide yes)
+			)
+		)
+		(pin "2"
+		)
+		(pin "1"
+		)
+		(instances
+			(project "PDB"
+				(path "/68b39743-cd9b-46b9-87c8-2ec94164be63"
+					(reference "R7")
+					(unit 1)
+				)

Commit message: Update Scheme
Parts:
- removed C3: CL05A105KA5NQNC (1uf ,0402 ,25v,X5R), easyeda2kicad:C0402, symbol easyeda2kicad:CL05A105KA5NQNC (1uf ,0402 ,25v,X5R)
- added C10, C3: CC0603KRX7R9BB104 (100nf , 0603 ,50v ,X7R), easyeda2kicad:C0603, symbol easyeda2kicad:CC0603KRX7R9BB104 (100nf , 0603 ,50v ,X7R)
- added C11, C12, C13, C14: CL10A225KA8NNNC, easyeda2kicad:C0603, symbol easyeda2kicad:CL10A225KA8NNNC (2.2uf , 0603 ,25v ,X5R)
- added C5, C6, C7: T521D107M025ATE040 (100uf , 7343 , 25v , tantalom), easyeda2kicad:CAP-SMD_L7.3-W4.3_H2.8, symbol easyeda2kicad:T521D107M025ATE040 (100uf , 7343 , 25v , tantalom)
- added C8, C9: CL10A106MA8NRNC (10uf , 0603 ,25v ,X5R), easyeda2kicad:C0603, symbol easyeda2kicad:CL10A106MA8NRNC (10uf , 0603 ,25v ,X5R)
- added R8: 0603WAF4423T5E, easyeda2kicad:R0603, symbol easyeda2kicad:0603WAF4423T5E (442kohm ,0603)
Connections:
- net 16.8V: now also U2.2 (VIN), C11.2, C12.2, C13.2, C14.2, R8.2
- net 16.8V_BAT: now also C4.1, C3.1, C5.1, C6.1, C7.1, C8.1, C9.1
- net GND: now also C4.2, CN1.1 (-), C11.1, C12.1, C13.1, C14.1, C3.2, C5.2, C6.2, C7.2, C8.2, C9.2
- net at U2.1 (BOOT): now also C10.1
- net at U2.8 (SW): now also C10.2
Other:
- moved on the sheet: C1, C2, C4, CN1, R1, R2, R3, R4, R5, R6, R7, U1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

Commit message: Update Scheme & DEV_DOC
Parts:
- removed R8: 0603WAF4423T5E, easyeda2kicad:R0603, symbol easyeda2kicad:0603WAF4423T5E (442kohm ,0603)
- added C15, C25: CL10B472KB8NNNC (4.7nF , 0603 ,50V ,X7R), easyeda2kicad:C0603, symbol easyeda2kicad:CL10B472KB8NNNC (4.7nF , 0603 ,50V ,X7R)
- added C16, C26: CL10C470JB8NNNC (47pF , 0603 ,50V ,C0G), easyeda2kicad:C0603, symbol easyeda2kicad:CL10C470JB8NNNC (47pF , 0603 ,50V ,C0G)
- added C17, C18, C19, C27, C28, C29: GRM21BR61A476ME15L (47uF , 0805 ,10V ,X5R), easyeda2kicad:C0805, symbol easyeda2kicad:GRM21BR61A476ME15L (47uF , 0805 ,10V ,X5R)
- added C20, C21, C22, C23: CL10A225KA8NNNC, easyeda2kicad:C0603, symbol easyeda2kicad:CL10A225KA8NNNC (2.2uf , 0603 ,25v ,X5R)
- added C24: CC0603KRX7R9BB104 (100nf , 0603 ,50v ,X7R), easyeda2kicad:C0603, symbol easyeda2kicad:CC0603KRX7R9BB104 (100nf , 0603 ,50v ,X7R)
- added D1, D2: B560C-13-F, easyeda2kicad:SMC_L7.1-W6.2-LS8.1-RD, symbol easyeda2kicad:B560C-13-F
- added R10, R16: 0603WAF2433T5E (243kohm , 0603), easyeda2kicad:R0603, symbol easyeda2kicad:0603WAF2433T5E (243kohm , 0603)
- added R11, R17: 0603WAF1692T5E (16.9kohm , 0603), easyeda2kicad:R0603, symbol easyeda2kicad:0603WAF1692T5E (16.9kohm , 0603)
- added R12, R19: 0603WAF1022T5E (10.2kohm , 0603), easyeda2kicad:R0603, symbol easyeda2kicad:0603WAF1022T5E (10.2kohm , 0603)
- added R13: 0603WAF5362T5E (53.6kohm , 0603), easyeda2kicad:R0603, symbol easyeda2kicad:0603WAF5362T5E (53.6kohm , 0603)
- added R14, R9: 0603WAF4423T5E, easyeda2kicad:R0603, symbol easyeda2kicad:0603WAF4423T5E (442kohm ,0603)
- added R15, R8: 0603WAF9092T5E (90.9kohm , 0603), easyeda2kicad:R0603, symbol easyeda2kicad:0603WAF9092T5E (90.9kohm , 0603)
- added R18: 0603WAF3162T5E (31.6kohm , 0603), easyeda2kicad:R0603, symbol easyeda2kicad:0603WAF3162T5E (31.6kohm , 0603)
- added U3: TPS54560DDAR, easyeda2kicad:SOIC-8_L5.0-W4.0-P1.27-LS6.0-BL-EP2.0, symbol easyeda2kicad:TPS54560DDAR
Connections:
- net 16.8V: now also C20.2, C21.2, C22.2, C23.2, R14.2, R9.2, U3.2 (VIN)
- net 3V3: now also C27.2, C28.2, C29.2, R18.2
- net GND: now also C15.1, C16.1, C17.1, C18.1, C19.1, C20.1, C21.1, C22.1, C23.1, C25.1, C26.1, C27.1, C28.1, C29.1, D1.2 (A), D2.2 (A), R10.1, R12.1, R15.1, R16.1, R19.1, R8.1, U3.7 (GND)
- net at U2.3 (EN): now also R8.2, R9.1
- net at U2.4 (RT/CLK): now also R10.2
- net FB: now reaches U2.5 (FB)
- net FB: now also R12.2, R13.1, R18.1, R19.2, U3.5 (FB)
- net at U2.6 (COMP): now also C16.2, R11.2
- new net: C15.2, R11.1
- new net: C25.2, R17.1
- new net: R14.1, R15.2, U3.3 (EN)
- new net: C24.1, U3.1 (BOOT)
- new net: R16.2, U3.4 (RT/CLK)
- new net: C26.2, R17.2, U3.6 (COMP)
- new net: C24.2, U3.8 (SW)
- new net 5V: C17.2, C18.2, C19.2, R13.2
Other:
- note added: "3V 4A"
- note added: "5V 5A"
- moved on the sheet: C10

Commit message: Update scheme & draw.io
Parts:
- removed R1: HOLR2725D-4W-0.5MR-1%, easyeda2kicad:R2725, symbol easyeda2kicad:HOLR2725D-4W-0.5MR-1%
- added C30: CL10A106KP8NNNC (10uf , 0603 ,10v,X5R), easyeda2kicad:C0603, symbol easyeda2kicad:CL10A106KP8NNNC (10uf , 0603 ,10v,X5R)
- added D3, D4: 603ESDA-05N (usb , esd , 0603), easyeda2kicad:D0603-BI, symbol easyeda2kicad:0603ESDA-05N (usb , esd , 0603)
- added Q1: DMG2301L-7, easyeda2kicad:SOT-23-3_L2.9-W1.3-P1.90-LS2.4-BR, symbol easyeda2kicad:DMG2301L-7
- added R1: HOLR2725D-4W-0.5MR-1% ( 0.5mohm , 2725), easyeda2kicad:R2725, symbol easyeda2kicad:HOLR2725D-4W-0.5MR-1% ( 0.5mohm , 2725)
- added R20, R21: 603WAF5101T5E (5.1kohm , 0603), easyeda2kicad:R0603, symbol easyeda2kicad:0603WAF5101T5E (5.1kohm , 0603)
- added SW1: JS102011JCQN (Slide Switch), easyeda2kicad:SW-SMD_JS102011JCQN, symbol easyeda2kicad:JS102011JCQN (Slide Switch)
- added U4, U5: LM74700QDBVRQ1, easyeda2kicad:SOT-23-6_L2.9-W1.6-P0.95-LS2.8-BL, symbol easyeda2kicad:LM74700QDBVRQ1
- added USB1: TYPE-C16PIN2MD(073) (USB TYPE C 16P), easyeda2kicad:USB-C-SMD_TYPE-C-6PIN-2MD-073, symbol easyeda2kicad:TYPE-C16PIN2MD(073) (USB TYPE C 16P)
Connections:
- net 16.8V: now also R1.2
- net 16.8V_BAT: now also R1.1
- net GND: now also CN1.3, CN1.4, C30.1, D3.1, D4.1, R20.1, R21.1, USB1.1 (GND), USB1.12 (GND), USB1.13 (SHELL), USB1.14 (SHELL)
- net FB renamed FB_3V3
- net FB_3V3: no longer R12.2, R13.1, U2.5 (FB)
- new net 16.8V_SW: SW1.3
- new net 5V_USB: C30.2, D3.2, D4.2, USB1.11 (VBUS), USB1.2 (VBUS)
- new net CC1: R21.2, USB1.4 (CC1)
- new net CC2: R20.2, USB1.10 (CC2)
- new net FB_5V: R12.2, R13.1, U2.5 (FB)
- no-connect marks 0 -> 7
Other:
- note added: "DC2DC 3V3"
- note added: "DC2DC 5V"
- note added: "ON/OFF SW"
- note added: "POWER FROM TYPE C"
- moved on the sheet: C10, C11, C12, C13, C14, C15, C16, C17, C18, C19, C20, C21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

Commit message: Update Scheme
Parts:
- removed Q1: DMG2301L-7, easyeda2kicad:SOT-23-3_L2.9-W1.3-P1.90-LS2.4-BR, symbol easyeda2kicad:DMG2301L-7
- added C31: CC0603KRX7R9BB104 (100nf , 0603 ,50v ,X7R), easyeda2kicad:C0603, symbol easyeda2kicad:CC0603KRX7R9BB104 (100nf , 0603 ,50v ,X7R)
- added Q2, Q3: AO3400A, easyeda2kicad:SOT-23-3_L2.9-W1.3-P1.90-LS2.4-BR, symbol easyeda2kicad:AO3400A
Connections:
- net 16.8V: now also Q2.2 (S); no longer C11.2, C12.2, C13.2, C14.2, C20.2, C21.2, C22.2, C23.2, R14.2, R9.2, U2.2 (VIN), U3.2 (VIN)
- net GND: now also U4.2 (GND), U5.2 (GND)
- net VOUT: now reaches U5.4 (CATHODE)
- net VOUT: now also C11.2, C12.2, C13.2, C14.2, C20.2, C21.2, C22.2, C23.2, R14.2, R9.2, U2.2 (VIN), U3.2 (VIN), U4.4 (CATHODE), Q2.3 (D), Q3.3 (D)
- net at U5.5 (GATE): now also Q3.1 (G)
- net at U4.5 (GATE): now also Q2.1 (G)
Other:
- moved on the sheet: U5

Commit message: Update Scheme
Parts:
- removed Q2, Q3: AO3400A, easyeda2kicad:SOT-23-3_L2.9-W1.3-P1.90-LS2.4-BR, symbol easyeda2kicad:AO3400A
- removed R14, R9: 0603WAF4423T5E, easyeda2kicad:R0603, symbol easyeda2kicad:0603WAF4423T5E (442kohm ,0603)
- removed R15, R8: 0603WAF9092T5E (90.9kohm , 0603), easyeda2kicad:R0603, symbol easyeda2kicad:0603WAF9092T5E (90.9kohm , 0603)
- added C32: CL21A226MAYNNNE (22uf , 0805 ,25v ,X5R), easyeda2kicad:C0805, symbol easyeda2kicad:CL21A226MAYNNNE (22uf , 0805 ,25v ,X5R)
- added C33, C34: CC0603KRX7R9BB104 (100nF , 0603 ,50V ,X7R), easyeda2kicad:C0603, symbol easyeda2kicad:CC0603KRX7R9BB104 (100nF , 0603 ,50V ,X7R)
- added C35: CC0603KRX7R9BB104 (100nf , 0603 ,50v ,X7R), easyeda2kicad:C0603, symbol easyeda2kicad:CC0603KRX7R9BB104 (100nf , 0603 ,50v ,X7R)
- added L1, L2: FXL1040-6R8-M, easyeda2kicad:IND-SMD_L11.5-W10.0_FXL1040, symbol easyeda2kicad:FXL1040-6R8-M
- added Q1, Q2: CSD18540Q5B(TOKMAS), easyeda2kicad:TDSON-8_L5.9-W5.2-P1.27-BL, symbol easyeda2kicad:CSD18540Q5B(TOKMAS)
Connections:
- net 16.8V: now also C31.2, U4.3 (EN), U4.6 (ANODE), C34.1, Q1.1 (S), Q1.2 (S), Q1.3 (S)
- net 3V3: now also L1.2
- net 5V: now also L2.2
- net 5V_USB: now also U5.3 (EN), U5.6 (ANODE), C33.1, C35.2, Q2.1 (S), Q2.2 (S), Q2.3 (S)
- net GND: now also C31.1, C32.1, C35.1
- net VOUT: now also SW1.2, U2.3 (EN), U3.3 (EN); no longer U4.4 (CATHODE), U5.4 (CATHODE)
- net at U5.1 (VCAP): now also C33.2
- net at U5.5 (GATE): now also Q2.4 (G)
- net at U4.5 (GATE): now also Q1.4 (G)
- net at C10.2, U2.8 (SW): now also D1.1 (K), L2.1
- net at D2.1 (K): now also C24.2, U3.8 (SW), L1.1
- net at U4.1 (VCAP): now also C34.2
- net 16.8V_SW renamed VOUT_SW
- net VOUT_SW: now also U4.4 (CATHODE), U5.4 (CATHODE), C32.2, Q1.5 (D), Q2.5 (D)
Other:
- moved on the sheet: C16, C31, R10, R16
