File: power_distribution_board/PDB.kicad_sch (KiCad schematic)
At the start: 68 parts, among them CN1 XT60PW-M, Q1 CSD18540Q5B(TOKMAS), Q2 CSD18540Q5B(TOKMAS), SW1 JS102011JCQN (Slide Switch), U1 INA226AIDGSR, U2 TPS54560DDAR, U3 TPS54560DDAR, U4 LM74700QDBVRQ1, U5 LM74700QDBVRQ1

Commit message: Update Scheme
Parts:
- added R8: 603WAF1002T5E (10kohm , 0603), easyeda2kicad:R0603, symbol easyeda2kicad:0603WAF1002T5E (10kohm , 0603)
- added U6: TL431_C5290159, easyeda2kicad:SOT-23-3_L2.9-W1.4-P1.90-LS2.6-BR, symbol easyeda2kicad:TL431_C5290159
- added U7: LM339DR, easyeda2kicad:SOIC-14_L8.7-W3.9-P1.27-LS6.0-BL, symbol easyeda2kicad:LM339DR

Commit message: Update scheme
Parts:
- added C36, C37: CC0603KRX7R9BB104 (100nf , 0603 ,50v ,X7R), easyeda2kicad:C0603, symbol easyeda2kicad:CC0603KRX7R9BB104 (100nf , 0603 ,50v ,X7R)
- added D5, D6: 603ESDA-05N (usb , esd , 0603), easyeda2kicad:D0603-BI, symbol easyeda2kicad:0603ESDA-05N (usb , esd , 0603)
- added H1, H2, H3, H4, H5, H6, H7, H8: MountingHole_Pad_MP, symbol Mechanical:MountingHole_Pad_MP
- added J2: CNJMA2012WV-S-10P, easyeda2kicad:CONN-SMD_10P-P2.00_CNJM_CNJMA2012WV-S-10P, symbol easyeda2kicad:CNJMA2012WV-S-10P
- added J4: HCZZ0494-4, easyeda2kicad:CONN-SMD_4P-P1.25_BM04B-GHS-TBT-LF-SN, symbol easyeda2kicad:HCZZ0494-4
- added LED1, LED2, LED3, LED4: 603Green509-620mcd (led green 0603), easyeda2kicad:LED0603-RD, symbol easyeda2kicad:KT-0603G (led green 0603)
- added R14, R28, R29, R30, R31: 0603WAF3301T5E (3.3kohm , 0603), easyeda2kicad:R0603, symbol easyeda2kicad:0603WAF3301T5E (3.3kohm , 0603)
- added R15: 0603WAF5492T5E (54.9kohm , 0603), easyeda2kicad:R0603, symbol easyeda2kicad:0603WAF5492T5E (54.9kohm , 0603)
- added R22, R24, R26: 603WAF1002T5E (10kohm , 0603), easyeda2kicad:R0603, symbol easyeda2kicad:0603WAF1002T5E (10kohm , 0603)
- added R23: 0603WAF5232T5E (52.3kohm , 0603), easyeda2kicad:R0603, symbol easyeda2kicad:0603WAF5232T5E (52.3kohm , 0603)
- added R25: RT0603BRD0750KL (50kohm , 0603), easyeda2kicad:R0603, symbol easyeda2kicad:RT0603BRD0750KL (50kohm , 0603)
- added R27: 0603WAF4752T5E (47.5kohm , 0603), easyeda2kicad:R0603, symbol easyeda2kicad:0603WAF4752T5E (47.5kohm , 0603)
- added R9: 603WAF0000T5E (0ohm , 0603), easyeda2kicad:R0603, symbol easyeda2kicad:0603WAF0000T5E (0ohm , 0603)
- added SW2: 6.0*6.0*6.0, easyeda2kicad:SW-SMD_4P-L6.0-W6.0-P4.50-LS8.6, symbol easyeda2kicad:6.0*6.0*6.0
- R2, R3: now not fitted; now left out of the parts list
- renumbered CN1 to J1, USB1 to J3
Connections:
- net 16.8V: now also H1.MP, H3.MP, H5.MP, H6.MP
- net 16.8V_BAT: now also SW2.1, SW2.2
- net 3V3: now also C37.2, J2.5, J2.6
- net 5V: now also C36.2, J2.1, J2.2
- net 5V_USB: now also J4.1
- net GND: now also R8.1, U6.3 (A), U7.12 (VCC-), C36.1, C37.1, D5.1, D6.1, H2.MP, H4.MP, H7.MP, H8.MP, J2.11, J2.12, J2.3, J2.4, J2.7, J2.8, J4.4, J4.5, J4.6, R22.1, R24.1, R26.1
- net SCL: now also J2.9
- net SDA: now also J2.10
- net at U6.1 (R): now also R9.1
- net 2.5V_REF: now reaches U6.2 (K)
- net 2.5V_REF: now also U7.11 (IN4+), U7.5 (IN2+), U7.7 (IN1+), U7.9 (IN3+), R14.2, R9.2
- net USB_D-: now reaches J3.5 (DN2)
- net USB_D-: now also J3.7 (DN1), D6.2, J4.2
- net USB_D+: now reaches J3.6 (DP1)
- net USB_D+: now also J3.8 (DP2), D5.2, J4.3
- net IN4-: now reaches R8.2
- net IN4-: now also U7.10 (IN4-), R15.1
- net at U7.1 (OUT1): now also LED3.1
- net at U7.13 (OUT4): now also LED2.1
- net at U7.14 (OUT3): now also LED1.1
- net at U7.2 (OUT2): now also LED4.1
- net 16.8V_BAT_M: now reaches U7.3 (VCC+)
- net 16.8V_BAT_M: now also R14.1, R15.2, R23.2, R25.2, R27.2, R28.2, R29.2, R30.2, R31.2, SW2.3, SW2.4
- net IN2-: now reaches U7.4 (IN2-)
- net IN2-: now also R22.2, R25.1
- net IN1-: now reaches U7.6 (IN1-)
- net IN1-: now also R26.2, R27.1
- net IN3-: now reaches U7.8 (IN3-)
- net IN3-: now also R23.1, R24.2
- new net: LED3.2, R30.1
- new net: LED2.2, R29.1
- new net: LED1.2, R28.1
- new net: LED4.2, R31.1
- no-connect marks 7 -> 3
Other:
- note added: "BATTERY 16.8V TO ESC"
- note added: "BATTERY 4S 16.8V INPUT"
- note added: "BATTERY INDICATOR"
- note added: "CONNECTORS FOR Flight Controller"
- note added: "CURRENT SENSOR"
- note added: "IDEAL DIODES"
- note added: "POWER & DATA FROM TYPE C"
- note removed: "POWER FROM TYPE C"
- moved on the sheet: C3, C30, C31, C32, C33, C34, C35, C4, C5, C6, C7, C8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

Commit message: Update Scheme 19/02/26
Parts:
- removed R4, R5: 603WAF0000T5E (0ohm , 0603), easyeda2kicad:R0603, symbol easyeda2kicad:0603WAF0000T5E (0ohm , 0603)
Connections:
- net 16.8V: now also C1.2, U1.9 (VIN-); no longer C34.1, U4.6 (ANODE)
- net 16.8V_BAT: now also C1.1, U1.10 (VIN+), U1.8 (VBUS)
- net 5V_USB: no longer C33.1, U5.6 (ANODE)
- net GND: now also U2.9 (EP), U3.9 (EP)
- new net: C34.1, U4.6 (ANODE)
- new net: C33.1, U5.6 (ANODE)

Commit message: routing in progress for PDB
Parts:
- removed D5, D6: 603ESDA-05N (usb , esd , 0603), easyeda2kicad:D0603-BI, symbol easyeda2kicad:0603ESDA-05N (usb , esd , 0603)
- removed H1, H2, H3, H4, H5, H6, H7, H8: MountingHole_Pad_MP, symbol Mechanical:MountingHole_Pad_MP
- removed SW2: 6.0*6.0*6.0, easyeda2kicad:SW-SMD_4P-L6.0-W6.0-P4.50-LS8.6, symbol easyeda2kicad:6.0*6.0*6.0
- added C38: CC0603KRX7R9BB104 (100nf , 0603 ,50v ,X7R), easyeda2kicad:C0603, symbol easyeda2kicad:CC0603KRX7R9BB104 (100nf , 0603 ,50v ,X7R)
- added H1, H2, H3, H4, H5, H6, H7, H8: TestPoint, TestPoint:TestPoint_THTPad_4.0x4.0mm_Drill2.0mm, symbol Connector:TestPoint
- added SW3: JS102011JCQN (Slide Switch), easyeda2kicad:SW-SMD_JS102011JCQN, symbol easyeda2kicad:JS102011JCQN (Slide Switch)
Connections:
- net 16.8V: now also C34.1, U1.8 (VBUS), U4.6 (ANODE), H1.1, H3.1, H5.1, H7.1
- net 16.8V_BAT: now also SW3.2; no longer U1.8 (VBUS)
- net 16.8V_BAT_M: now also SW3.3
- net 3V3: now also C38.2
- net 5V_USB: now also C33.1, U5.6 (ANODE)
- net GND: now also C38.1, H2.1, H4.1, H6.1, H8.1
Other:
- note added: "BATTERY INDICATOR SWITCH"
