File: power_distribution_board/PDB.kicad_pcb (KiCad board)
At the start: 6 copper layers, 50 x 50 mm, 98 parts, among them J1 XT60PW-M, J2 CNJMA2012WV-S-10P, J3 TYPE-C16PIN2MD(073) (USB TYPE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, J4 HCZZ0494-4, Q1 CSD18540Q5B(TOKMAS), Q2 CSD18540Q5B(TOKMAS), SW1 JS102011JCQN (Slide Switch), SW3 JS102011JCQN (Slide Switch), U1 INA226AIDGSR, U2 TPS54560DDAR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

Commit message: Finished routing of PDB
Parts:
- moved R10 2.96 mm to (141.1, 112.4)
- moved R16 2.05 mm to (156.5, 116.8)
- moved D2 1.59 mm to (147.0, 104.8)
- moved R17 1.07 mm to (141.9, 115.7)
- moved C10 0.96 mm to (141.3, 106.4)
- moved C13 0.24 mm to (142.0, 109.3)
- moved C24 0.12 mm to (154.1, 110.0)
Routing:
- net VOUT_SW: track 72.0 -> 39.1 mm
- net Net-(D2-K): track 0.00 -> 25.0 mm, vias 0 -> 4
- net /FB_3V3: track 0.00 -> 15.6 mm, vias 0 -> 3
- net Net-(U3-COMP): track 0.00 -> 6.18 mm, vias 0 -> 3
- net Net-(U2-RT/CLK): track 0.00 -> 2.91 mm
- net Net-(C25-Pad2): track 0.00 -> 2.85 mm, vias 0 -> 2
- net Net-(U3-RT/CLK): track 0.00 -> 2.75 mm
- net Net-(U3-BOOT): track 0.00 -> 1.48 mm
- net Net-(D1-K): track 25.6 -> 26.6 mm
- net Net-(U2-BOOT): track 3.67 -> 4.38 mm
- net GND: track 18.3 -> 18.8 mm, vias 56 -> 63
- net VOUT: vias 5 -> 6

Commit message: Finished PDB
Parts:
- added G***: LOGO, easyeda2kicad:LAMPEL_pdb_LOGO, B.Cu at (161.7, 101.8)
- moved C3 1.43 mm to (158.3, 86.9)
- moved C10 1.41 mm to (141.4, 105.0)
- moved C24 1.28 mm to (155.4, 110.0), turned to 0 degrees
- moved C31 1.00 mm to (165.6, 98.8)
- moved R26 0.80 mm to (127.0, 95.1)
- moved C33 0.63 mm to (160.2, 114.5)
- moved U5 0.40 mm to (160.1, 117.3)
- moved R28 0.40 mm to (126.8, 85.8)
- moved C8 0.36 mm to (159.6, 90.6)
- moved R27 0.35 mm to (128.8, 95.1)
- moved C9 0.10 mm to (159.6, 88.7)
- moved R25 0.05 mm to (130.6, 95.1)
Routing:
- net GND: track 18.8 -> 23.3 mm, vias 63 -> 64
- net VOUT_SW: track 39.1 -> 37.1 mm
- net 5V_USB: track 19.8 -> 18.4 mm
- net /USB_D-: track 17.2 -> 18.5 mm
- net Net-(D1-K): track 26.6 -> 27.8 mm
- net /FB_3V3: track 15.6 -> 14.5 mm
- net Net-(U3-BOOT): track 1.48 -> 2.49 mm
- net Net-(U2-BOOT): track 4.38 -> 5.34 mm
- net Net-(U5-VCAP): track 1.23 -> 2.06 mm
- net /IN1-: track 4.11 -> 4.91 mm
- net /IN2-: track 11.0 -> 10.3 mm
- net 16.8V_BAT: vias 16 -> 15
- added copper zone on In2.Cu, net 16.8V
- added copper zone on F.Cu, net 16.8V_BAT
- added copper zone on In4.Cu, net 16.8V_BAT
- added copper zone on F.Cu, net 16.8V_BAT_M
- added copper zone on F.Cu, net 3V3
- added copper zone on In2.Cu, net 3V3
- added copper zone on F.Cu, net Net-(D1-K)
- added copper zone on In4.Cu, net Net-(D2-K)
- added copper zone on In2.Cu, net VOUT_SW
Other:
- board text added: "PDB V1.0 Eli Yakubov Eyal Lampel"
