File: flight_controller/STM32H7.kicad_sch (KiCad schematic)
At the start: 48 parts, among them SW2 6.0*6.0*6.0, U1 STM32H743IIT6, U6 HB-PH9-12727PB2GOB, X1 SC-32S32.768kHz20PPM7pF, X2 X322525MOB4SI

Commit message: Schematic complete, ready for layout. Added USB, TPs, power conn, updated clocks, ran Rules Checker and general review
Parts:
- removed C10, C9: 0603CG7R0C500NT (7pf , 0603 , 50v), easyeda2kicad:C0603, symbol lampelKicadLIB:0603CG7R0C500NT (7pf , 0603 , 50v)
- removed C51, C52: CL10C120JB8NNNC ( 12pf , 0603 , 50v , C0G), easyeda2kicad:C0603, symbol lampelKicadLIB:CL10C120JB8NNNC ( 12pf , 0603 , 50v , C0G)
- removed D10: KT-0603R, easyeda2kicad:LED0603-RD, symbol easyeda2kicad:KT-0603R
- removed D3: 0603 Green 509-620mcd, easyeda2kicad:LED0603-RD, symbol easyeda2kicad:0603Green509-620mcd
- removed R5, R50: 603WAF1000T5E (100ohm , 0603), easyeda2kicad:R0603, symbol lampelKicadLIB:0603WAF1000T5E (100ohm , 0603)
- removed X1: SC-32S32.768kHz20PPM7pF, easyeda2kicad:OSC-SMD_L3.2-W1.5, symbol lampelKicadLIB:SC-32S32.768kHz20PPM7pF
- removed X2: X322525MOB4SI, easyeda2kicad:CRYSTAL-SMD_4P-L3.2-W2.5-BL, symbol lampelKicadLIB:X322525MOB4SI
- added C1, C10, C2, C51: CC0603JRNPO9BN100 (10pF , 0603 ,50V ,X7R), easyeda2kicad:C0603, symbol lampelKicadLIB:CC0603JRNPO9BN100 (10pF , 0603 ,50V ,X7R)
- added C9: CC0603KRX7R9BB104 (100nf , 0603 ,50v ,X7R), easyeda2kicad:C0603, symbol lampelKicadLIB:CC0603KRX7R9BB104 (100nf , 0603 ,50v ,X7R)
- added D12: KT-0603R, easyeda2kicad:LED0603-RD, symbol easyeda2kicad:KT-0603R
- added D5: 0603 Green 509-620mcd, easyeda2kicad:LED0603-RD, symbol easyeda2kicad:0603Green509-620mcd
- added R106, R107: 0603WAF1002T5E, easyeda2kicad:R0603, symbol easyeda2kicad:0603WAF1002T5E
- added R5, R7: 603WAF0000T5E (0ohm , 0603), easyeda2kicad:R0603, symbol lampelKicadLIB:0603WAF0000T5E (0ohm , 0603)
- added R58, R59: 603WAF1000T5E (100ohm , 0603), easyeda2kicad:R0603, symbol lampelKicadLIB:0603WAF1000T5E (100ohm , 0603)
- added TP10, TP11, TP12, TP13, TP14, TP3, TP4, TP6, TP7, TP8, TP9: TestPoint, TestPoint:TestPoint_Pad_2.0x2.0mm, symbol Connector:TestPoint
- added X1: XKXEL89CLI-SUAYLC-32.768K, easyeda2kicad:OSC-SMD_2P-L3.2-W1.5, symbol lampelKicadLIB:XKXEL89CLI-SUAYLC-32.768K
- added X2: XL2EL89CLI-111YLC-16M, easyeda2kicad:CRYSTAL-SMD_4P-L3.2-W2.5-BL, symbol lampelKicadLIB:XL2EL89CLI-111YLC-16M
- R27, R28: now not fitted; now left out of the parts list
Connections:
- net SPI6_SCK is gone; now on net FMU_SWO: U1.161 (PB3)
- net SWCLK is gone; now on net FMU_SWCLK: U6.6
- net SWDIO is gone; now on net FMU_SWDIO: U6.4
- net 3V3: now also C9.2, D12.2 (A), D5.2 (A), R106.2, R107.2, R7.2
- net ADC1_IN16: now also TP7.1
- net ADC1_INP18: now also TP8.1
- net ADC1_INP5: now also TP10.1
- net ADC1_INP9: now also TP9.1
- net ADC3_INP0: now also TP11.1
- net ADC3_INP1: now also TP12.1
- net FMU_CAP1: now also TP14.1
- net GND: now also C1.1, C10.1, C2.1, C51.1, C9.1, R5.1, X2.2 (GND), X2.4 (GND)
- net I2C4_SCL: now also R106.1
- net I2C4_SDA: now also R107.1
- net NFC_GPIO: now also TP13.1
- net OSC32_IN: now also C10.2, X1.1
- net OSC32_OUT: now also C51.2, X1.2
- net OSC_IN: now also C2.2, X2.1
- net OSC_OUT: now also C1.2, X2.3
- net TIM2_CH3_HEATER: now also TP3.1
- net VCAP1: now also TP4.1
- net nARMED: now also TP3.1
- net nPOWER_IN_A: now also TP6.1
- net FMU_SWO: now reaches U6.8
- net I2C2_DRDY1: now reaches U1.109 (PG5)
- net PDR_ON: now reaches U1.171 (PDR_ON)
- net PDR_ON: now also R5.2, R7.1
- net ETH_POWER_EN renamed ETH_NRST
- net nLED_GREEN renamed FMU_LED1_GREEN
- net FMU_LED1_GREEN: now also R58.2
- net nLED_RED renamed FMU_LED2_RED
- net FMU_LED2_RED: now also R59.2
- net nPOWER_IN_B renamed PWR_GPIO1
- new net: D5.1 (K), R58.1
- new net: D12.1 (K), R59.1
- no-connect marks 5 -> 35
Other:
- note added: "C_ext = 2*(C_load - C_stray) = 2*(9 - 4) = 10pF"
- note added: "Crystal 16MHz"
- note added: "Crystal 32.768kHz"
- note added: "VCP"
- note added: "was SPI6_SCK"
- note removed: "SWO"
- moved on the sheet: C15, C16, C3, C4

Commit message: Started the placement process
Parts:
- added TP11: TestPoint, TestPoint:TestPoint_Pad_2.0x2.0mm, symbol Connector:TestPoint
- renumbered C10 to C1, C27 to C10, C26 to C11, C25 to C12, C24 to C13, C23 to C14, C22 to C15, C21 to C16, C20 to C17, C6 to C18, C5 to C19, C51 to C2, C11 to C20, C12 to C21, C13 to C22, C14 to C23, C9 to C24, C15 to C25, C4 to C26, C16 to C27, C3 to C28, C1 to C3, C2 to C4, C32 to C5, C31 to C6, C30 to C7, C29 to C8, C28 to C9, D5 to D1, D12 to D2, R68 to R1, R5 to R10, R73 to R11, R2 to R12, R58 to R13, R59 to R14, R1 to R15, R6 to R16, R28 to R17, R27 to R18, R66 to R2, R70 to R3, R106 to R4, R69 to R5, R67 to R6, R71 to R7, R107 to R8, R7 to R9, SW2 to SW1, TP3 to TP1, TP14 to TP10, TP4 to TP12, TP13 to TP2, TP11 to TP3, TP12 to TP4, TP7 to TP5, TP8 to TP6, TP9 to TP7, TP10 to TP8, TP6 to TP9, U6 to U1, U1 to U2
Connections:
- net TIM2_CH3_HEATER: now also TP11.1; no longer TP1.1

Commit message: Finished placement
Connections:
- net USB_OTG_FS_DM renamed USB_OTG_FS_D-
- net USB_OTG_FS_DP renamed USB_OTG_FS_D+
Changed lines of the file:
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@@
 		)
 	)
-	(label "USB_OTG_FS_DP"
+	(label "USB_OTG_FS_D+"
 		(at 488.95 143.51 0)
 		(effects
@@
 		)
 	)
-	(label "USB_OTG_FS_DM"
+	(label "USB_OTG_FS_D-"
 		(at 488.95 146.05 0)
 		(effects
@@
 		)
 	)
-	(hierarchical_label "USB_OTG_FS_DM"
+	(hierarchical_label "USB_OTG_FS_D-"
 		(shape bidirectional)
 		(at 511.81 146.05 0)
@@
 		)
 	)
-	(hierarchical_label "USB_OTG_FS_DP"
+	(hierarchical_label "USB_OTG_FS_D+"
 		(shape bidirectional)
 		(at 511.81 143.51 0)
