File: flight_controller/STM32H7.kicad_sch (KiCad schematic)
At the start: 65 parts, among them SW1 6.0*6.0*6.0, U1 HB-PH9-12727PB2GOB, U2 STM32H743IIT6, X1 XKXEL89CLI-SUAYLC-32.768K, X2 XL2EL89CLI-111YLC-16M

Commit message: renamed some connectors to j instead of cn
Parts:
- renumbered U1 to J22
Connections:
- net PWR_GPIO1 renamed nPOWER_IN_B
- no-connect marks 35 -> 36
Changed lines of the file:
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@@
 	)
 	(no_connect
+		(at 511.81 186.69)
+	)
+	(no_connect
 		(at 290.83 151.13)
 	)
@@
 	(wire
 		(pts
-			(xy 486.41 186.69) (xy 511.81 186.69)
-		)
-		(stroke
-			(width 0)
-			(type default)
-		)
-	)
-	(wire
-		(pts
 			(xy 486.41 229.87) (xy 511.81 229.87)
 		)
@@
 	(wire
 		(pts
+			(xy 486.41 186.69) (xy 511.81 186.69)
+		)
+		(stroke
+			(width 0)
+			(type default)
+		)
+	)
+	(wire
+		(pts
 			(xy 290.83 204.47) (xy 316.23 204.47)
 		)
@@
 		)
 	)
-	(label "PWR_GPIO1"
+	(label "nPOWER_IN_B"
 		(at 488.95 186.69 0)
 		(effects
@@
 		)
 	)
-	(hierarchical_label "PWR_GPIO1"
-		(shape input)
-		(at 511.81 186.69 0)
-		(effects
-			(font
-				(size 1.27 1.27)
-			)
-			(justify left)
-		)
-	)
 	(hierarchical_label "FMU_CH1"
 		(shape output)
@@
 		(on_board yes)
 		(dnp no)
-		(property "Reference" "U1"
+		(property "Reference" "J22"
 			(at 288.29 337.82 0)
 			(effects
@@
 			(project "FP_BOARD"
 				(path "/17737359-1a8e-4237-8899-d9604030bc1d/21c4e215-368e-4a6b-9b68-3566112ef4e7"
-					(reference "U1")
+					(reference "J22")
 					(unit 1)
 				)
