File: flight_controller/CAN_and_External.kicad_sch (KiCad schematic)
At the start: 22 parts, among them J1 HCZZ0494-4, J11 A1257WV-S-6P-LCP, J18 A1257WV-S-6P-LCP, J2 HCZZ0494-4, J8 SM04B-SRSS-TB(LF)(SN), U13 TJA1051T/3/1J, U9 TJA1051T/3/1J

Commit message: Started the placement process
Parts:
- renumbered C67 to C39, C19 to C40, C18 to C41, C46 to C42, C39 to C43, C56 to C44, C74 to C45, J8 to J5, J11 to J6, J1 to J7, J2 to J8, J18 to J9, R94 to R42, R95 to R43, R62 to R44, R63 to R45, R64 to R46, R65 to R47, R44 to R48, R45 to R49, U13 to U7, U9 to U8

Commit message: Updated power and usb connectors, annotations and netlist check
Parts:
- renumbered J8 to J10, J9 to J11, J5 to J7, J6 to J8, J7 to J9, U7 to U4, U8 to U5
Changed lines of the file:
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@@
 		(dnp no)
 		(fields_autoplaced yes)
-		(property "Reference" "J9"
+		(property "Reference" "J11"
 			(at 442.468 280.416 0)
 			(do_not_autoplace yes)
@@
 			(project "FP_BOARD"
 				(path "/17737359-1a8e-4237-8899-d9604030bc1d/bc534bd1-f491-4966-ba4f-9fc6d85cb066"
-					(reference "J9")
+					(reference "J11")
 					(unit 1)
 				)
@@
 		(dnp no)
 		(fields_autoplaced yes)
-		(property "Reference" "J8"
+		(property "Reference" "J10"
 			(at 342.392 162.814 0)
 			(do_not_autoplace yes)
@@
 			(project "FP_BOARD"
 				(path "/17737359-1a8e-4237-8899-d9604030bc1d/bc534bd1-f491-4966-ba4f-9fc6d85cb066"
-					(reference "J8")
+					(reference "J10")
 					(unit 1)
 				)
@@
 		(dnp no)
 		(fields_autoplaced yes)
-		(property "Reference" "U8"
+		(property "Reference" "U5"
 			(at 250.19 86.36 0)
 			(effects
@@
 			(project "FP_BOARD"
 				(path "/17737359-1a8e-4237-8899-d9604030bc1d/bc534bd1-f491-4966-ba4f-9fc6d85cb066"
-					(reference "U8")
+					(reference "U5")
 					(unit 1)
 				)
@@
 		(dnp no)
 		(fields_autoplaced yes)
-		(property "Reference" "U7"
+		(property "Reference" "U4"
 			(at 248.92 156.21 0)
 			(effects
@@
 			(project "FP_BOARD"
 				(path "/17737359-1a8e-4237-8899-d9604030bc1d/bc534bd1-f491-4966-ba4f-9fc6d85cb066"
-					(reference "U7")
+					(reference "U4")
 					(unit 1)
 				)
@@
 		(on_board yes)
 		(dnp no)
-		(property "Reference" "J5"
+		(property "Reference" "J7"
 			(at 158.75 275.59 90)
 			(effects
@@
 			(project "FP_BOARD"
 				(path "/17737359-1a8e-4237-8899-d9604030bc1d/bc534bd1-f491-4966-ba4f-9fc6d85cb066"
-					(reference "J5")
+					(reference "J7")
 					(unit 1)
 				)
@@
 		(dnp no)
 		(fields_autoplaced yes)
-		(property "Reference" "J7"
+		(property "Reference" "J9"
 			(at 342.392 92.964 0)
 			(do_not_autoplace yes)
@@
 			(project "FP_BOARD"
 				(path "/17737359-1a8e-4237-8899-d9604030bc1d/bc534bd1-f491-4966-ba4f-9fc6d85cb066"
-					(reference "J7")
+					(reference "J9")
 					(unit 1)
 				)
@@
 		(dnp no)
 		(fields_autoplaced yes)
-		(property "Reference" "J6"
+		(property "Reference" "J8"
 			(at 316.738 276.606 0)
 			(do_not_autoplace yes)
@@
 			(project "FP_BOARD"
 				(path "/17737359-1a8e-4237-8899-d9604030bc1d/bc534bd1-f491-4966-ba4f-9fc6d85cb066"
-					(reference "J6")
-					(unit 1)
-				)
+					(reference "J8")
+					(unit 1)
+				)

Commit message: Revert to state of commit 2458262 moved all to components to top
Reverts commits: d012532, 3d9c600, 58bc0ac
Parts:
- renumbered J7 to J5, J8 to J6, J9 to J7, J10 to J8, J11 to J9, U4 to U7, U5 to U8
Changed lines of the file:
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@@
 		(dnp no)
 		(fields_autoplaced yes)
-		(property "Reference" "J11"
+		(property "Reference" "J9"
 			(at 442.468 280.416 0)
 			(do_not_autoplace yes)
@@
 			(project "FP_BOARD"
 				(path "/17737359-1a8e-4237-8899-d9604030bc1d/bc534bd1-f491-4966-ba4f-9fc6d85cb066"
-					(reference "J11")
+					(reference "J9")
 					(unit 1)
 				)
@@
 		(dnp no)
 		(fields_autoplaced yes)
-		(property "Reference" "J10"
+		(property "Reference" "J8"
 			(at 342.392 162.814 0)
 			(do_not_autoplace yes)
@@
 			(project "FP_BOARD"
 				(path "/17737359-1a8e-4237-8899-d9604030bc1d/bc534bd1-f491-4966-ba4f-9fc6d85cb066"
-					(reference "J10")
+					(reference "J8")
 					(unit 1)
 				)
@@
 		(dnp no)
 		(fields_autoplaced yes)
-		(property "Reference" "U5"
+		(property "Reference" "U8"
 			(at 250.19 86.36 0)
 			(effects
@@
 			(project "FP_BOARD"
 				(path "/17737359-1a8e-4237-8899-d9604030bc1d/bc534bd1-f491-4966-ba4f-9fc6d85cb066"
-					(reference "U5")
+					(reference "U8")
 					(unit 1)
 				)
@@
 		(dnp no)
 		(fields_autoplaced yes)
-		(property "Reference" "U4"
+		(property "Reference" "U7"
 			(at 248.92 156.21 0)
 			(effects
@@
 			(project "FP_BOARD"
 				(path "/17737359-1a8e-4237-8899-d9604030bc1d/bc534bd1-f491-4966-ba4f-9fc6d85cb066"
-					(reference "U4")
+					(reference "U7")
 					(unit 1)
 				)
@@
 		(on_board yes)
 		(dnp no)
-		(property "Reference" "J7"
+		(property "Reference" "J5"
 			(at 158.75 275.59 90)
 			(effects
@@
 			(project "FP_BOARD"
 				(path "/17737359-1a8e-4237-8899-d9604030bc1d/bc534bd1-f491-4966-ba4f-9fc6d85cb066"
-					(reference "J7")
+					(reference "J5")
 					(unit 1)
 				)
@@
 		(dnp no)
 		(fields_autoplaced yes)
-		(property "Reference" "J9"
+		(property "Reference" "J7"
 			(at 342.392 92.964 0)
 			(do_not_autoplace yes)
@@
 			(project "FP_BOARD"
 				(path "/17737359-1a8e-4237-8899-d9604030bc1d/bc534bd1-f491-4966-ba4f-9fc6d85cb066"
-					(reference "J9")
+					(reference "J7")
 					(unit 1)
 				)
@@
 		(dnp no)
 		(fields_autoplaced yes)
-		(property "Reference" "J8"
+		(property "Reference" "J6"
 			(at 316.738 276.606 0)
 			(do_not_autoplace yes)
@@
 			(project "FP_BOARD"
 				(path "/17737359-1a8e-4237-8899-d9604030bc1d/bc534bd1-f491-4966-ba4f-9fc6d85cb066"
-					(reference "J8")
-					(unit 1)
-				)
+					(reference "J6")
+					(unit 1)
+				)

Commit message: Advanced in routing
Parts:
- added C79, C80: CC0603KRX7R9BB104 (100nf , 0603 ,50v ,X7R), easyeda2kicad:C0603, symbol lampelKicadLIB:CC0603KRX7R9BB104 (100nf , 0603 ,50v ,X7R)
Connections:
- net 5V: now also C79.2, C80.2
- net GND: now also C79.1, C80.1
