File: flight_controller/FP_BOARD.kicad_pcb (KiCad board)
At the start: 6 copper layers, 100 x 100 mm, 246 parts, among them J1 HX PZ2.54-3X4P ZZ, J10 CNJMA2012WV-S-10P, J11 A1257WV-S-6P-LCP, J12 A1257WV-S-6P-LCP, J13 A1257WV-S-6P-LCP, J14 HR911105A_C12074, J15 A1257WV-S-6P-LCP, J16 HCZZ0494-2, J17 HCZZ0494-4, J18 A1251WV-S-4P, J19 A1251WV-S-6P, J2 B3B-ZR-SM4-TF(LF)(SN), J20 A1251WV-S-3P, J21 HB-PH9-12727PB2GOB, J22 HB-PH9-12727PB2GOB, J3 HX PZ2.54-3X4P ZZ, J4 HX PZ2.54-3X4P ZZ, J5 SM04B-SRSS-TB(LF)(SN), J6 A1257WV-S-6P-LCP, J7 HCZZ0494-4, J8 HCZZ0494-4, J9 A1257WV-S-6P-LCP, Q1 AO3400A, SW1 6.0*6.0*6.0, SW2 6.0*6.0*6.0, U10 24LC64-I/SN, U11 FM25V02A-GTR, U12 MPU6500, U13 MS561101BA03-50, U14 LAN8742AI-CZ, U15 SN74LVC1G07DBVR_C19829659, U2 STM32H743IIT6, U4 STM32F103C8T6, U5 SN74LVC2G240DCTR, U56 ICM-20689, U7 TJA1051T/3/1J, U8 TJA1051T/3/1J, U9 W25Q512JVFIQ, X1 XKXEL89CLI-SUAYLC-32.768K, X2 XL2EL89CLI-111YLC-16M, X3 X322524MLB4SI_C5210646, X4 XL2EL89CMI-111YLC-25M

Commit message: Advanced in routing
Parts:
- removed Card1: TFPUSH (Micro SD card), easyeda2kicad:TF-SMD_TF-PUSH
- added C78: GRM21BR61A476ME15L (47uF , 0805 ,10V ,X5R), easyeda2kicad:C0805, F.Cu at (168.5, 122.1)
- added C79: CC0603KRX7R9BB104 (100nf , 0603 ,50v ,X7R), easyeda2kicad:C0603, F.Cu at (93.7, 73.9)
- added C80: CC0603KRX7R9BB104 (100nf , 0603 ,50v ,X7R), easyeda2kicad:C0603, F.Cu at (94.0, 61.2)
- added C81: GRM21BR61A476ME15L (47uF , 0805 ,10V ,X5R), easyeda2kicad:C0805, F.Cu at (154.9, 122.1)
- added C82: CC0603KRX7R9BB104 (100nf , 0603 ,50v ,X7R), easyeda2kicad:C0603, F.Cu at (139.2, 42.0)
- added Card2: TF-01A, easyeda2kicad:TF-SMD_TF-01A, F.Cu at (95.8, 113.4)
- moved R32 45.7 mm to (159.6, 94.3), turned to 0 degrees
- moved SW1 15.4 mm to (166.3, 107.2), turned to 0 degrees
- moved C33 13.9 mm to (168.4, 59.8), turned to 90 degrees
- moved R40 13.5 mm to (159.4, 79.2)
- moved R39 13.2 mm to (159.0, 77.3)
- moved R27 12.1 mm to (156.3, 70.7)
- moved R28 12.1 mm to (159.5, 70.6)
- moved R29 11.7 mm to (156.7, 74.8)
- moved R30 11.7 mm to (159.4, 74.7)
- moved R8 11.3 mm to (179.9, 123.8)
- moved TP9 11.3 mm to (140.4, 82.2)
- moved R35 10.6 mm to (159.9, 81.6)
- moved R36 10.5 mm to (159.9, 84.2)
- moved J3 10.5 mm to (166.8, 85.5)
- moved R37 10.5 mm to (159.8, 86.7)
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Routing:
- net GND: track 14.0 -> 247.1 mm, vias 9 -> 209
- net 3V3: track 0.00 -> 125.1 mm, vias 0 -> 47
- net /USB_OTG_FS_D+: track 0.00 -> 43.7 mm
- net /USB_OTG_FS_D-: track 0.00 -> 43.7 mm
- net 5V: track 8.71 -> 44.2 mm, vias 0 -> 12
- net /ETH_MDC: track 0.00 -> 28.9 mm, vias 0 -> 2
- net /ETH/ETH_TXP: track 0.00 -> 23.4 mm, vias 0 -> 1
- net /USB/USB_5V: track 0.00 -> 19.8 mm
- net /USB_OTG_FS_VBUS: track 0.00 -> 14.2 mm
- net Net-(J14-Pad11): track 0.00 -> 8.24 mm
- net Net-(U7-CANL): track 0.00 -> 7.60 mm
- net Net-(U7-CANH): track 0.00 -> 7.57 mm
- net Net-(Q1-G): track 0.00 -> 7.12 mm
- net Net-(J14-Pad10): track 0.00 -> 6.95 mm
- net Net-(D5-A): track 0.00 -> 6.17 mm
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- added copper zone on In2.Cu, net 3V3
- added copper zone on In4.Cu, net 5V
- added copper zone on B.Cu, net GND
- added copper zone on In1.Cu, net GND
- added copper zone on In3.Cu, net GND

Commit message: Advanced in routing more
Parts:
- moved C37 3.48 mm to (146.9, 47.6), turned to -90 degrees
- moved C79 2.04 mm to (94.0, 71.8)
- moved C44 1.64 mm to (107.5, 40.2)
- moved C39 1.37 mm to (93.9, 43.4), turned to -90 degrees
- moved C38 1.19 mm to (94.4, 39.7)
- moved C18 1.11 mm to (151.1, 92.0), turned to 90 degrees
- moved C32 0.81 mm to (164.9, 45.8)
- moved C76 0.81 mm to (178.4, 120.7)
- moved R48 0.77 mm to (95.9, 69.1)
- moved C42 0.77 mm to (99.5, 53.7), turned to 180 degrees
- moved C77 0.75 mm to (135.1, 55.6)
- moved C31 0.71 mm to (174.2, 49.7), turned to 90 degrees
- moved C73 0.64 mm to (129.5, 39.4)
- moved C19 0.61 mm to (128.1, 98.5)
- moved C13 0.61 mm to (120.1, 85.1)
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Routing:
- net GND: track 247.1 -> 175.6 mm, vias 209 -> 261
- net 3V3: track 125.1 -> 89.7 mm, vias 47 -> 67
- net 5V: track 44.2 -> 28.0 mm, vias 12 -> 27
- net Net-(U4-PB2): track 0.00 -> 4.38 mm

Commit message: Started critical lines routing
Parts:
- moved R78 4.43 mm to (113.2, 110.5)
- moved R80 4.31 mm to (113.8, 106.0)
- moved R13 3.98 mm to (116.5, 100.8)
- moved D1 3.75 mm to (112.7, 100.8)
- moved R99 2.73 mm to (131.8, 108.1)
- moved R14 1.75 mm to (122.1, 97.0)
- moved C49 0.91 mm to (103.4, 111.7)
- moved C80 0.40 mm to (93.6, 60.9)
- moved R12 0.38 mm to (143.3, 53.8), turned to 180 degrees
- moved C45 0.36 mm to (93.8, 102.0)
- moved C79 0.28 mm to (93.7, 71.8)
Routing:
- net /ETH_TX_EN: track 0.00 -> 49.3 mm
- net /ETH_MDIO: track 0.00 -> 43.4 mm
- net /ETH/ETH_LED1: track 0.00 -> 33.7 mm
- net /ETH_TXD1: track 0.00 -> 32.9 mm
- net /ETH_TXD0: track 0.00 -> 31.6 mm
- net GND: track 175.6 -> 144.4 mm, vias 261 -> 271
- net /ETH/ETH_TXP: track 23.4 -> 3.88 mm
- net /ETH/ETH_RXN: track 0.00 -> 11.7 mm, vias 0 -> 1
- net /ETH/ETH_RXP: track 0.00 -> 7.61 mm
- net /ETH/ETH_TXN: track 0.00 -> 6.72 mm, vias 0 -> 1
- net 5V: track 28.0 -> 23.7 mm, vias 27 -> 28
- net /ETH_NRST: track 0.00 -> 3.42 mm
- net /ETH/ETH_LED2: track 0.00 -> 3.00 mm
- net 3V3: track 89.7 -> 89.1 mm
