File: flight_controller/FP_BOARD.kicad_pcb (KiCad board)
At the start: 6 copper layers, 100 x 100 mm, 249 parts, among them J1 HX PZ2.54-3X4P ZZ, J10 CNJMA2012WV-S-10P, J11 A1257WV-S-6P-LCP, J12 A1257WV-S-6P-LCP, J13 A1257WV-S-6P-LCP, J14 HR911105A_C12074, J15 A1257WV-S-6P-LCP, J16 HCZZ0494-2, J17 HCZZ0494-4, J18 A1251WV-S-4P, J19 A1251WV-S-6P, J2 B3B-ZR-SM4-TF(LF)(SN), J20 A1251WV-S-3P, J21 HB-PH9-12727PB2GOB, J22 HB-PH9-12727PB2GOB, J3 HX PZ2.54-3X4P ZZ, J4 HX PZ2.54-3X4P ZZ, J5 SM04B-SRSS-TB(LF)(SN), J6 A1257WV-S-6P-LCP, J7 HCZZ0494-4, J8 HCZZ0494-4, J9 A1257WV-S-6P-LCP, Q1 AO3400A, SW1 6.0*6.0*6.0, SW2 6.0*6.0*6.0, U10 24LC64-I/SN, U11 FM25V02A-GTR, U12 MPU6500, U13 MS561101BA03-50, U14 LAN8742AI-CZ, U15 SN74LVC1G07DBVR_C19829659, U2 STM32H743IIT6, U4 STM32F103C8T6, U5 SN74LVC2G240DCTR, U56 ICM-20689, U7 TJA1051T/3/1J, U8 TJA1051T/3/1J, U9 W25Q512JVFIQ, X1 XKXEL89CLI-SUAYLC-32.768K, X2 XL2EL89CLI-111YLC-16M, X3 X322524MLB4SI_C5210646, X4 XL2EL89CMI-111YLC-25M

Commit message: Router a bit more
Routing:
- net /UART2_RTS_TELEM3: track 0.00 -> 75.2 mm, vias 0 -> 2
- net /UART2_TX_TELEM3: track 0.00 -> 69.8 mm, vias 0 -> 2
- net /UART2_CTS_TELEM3: track 0.00 -> 55.9 mm, vias 0 -> 3
- net /STM32F1/USART6_TX_TO_IO-NC: track 0.00 -> 53.5 mm, vias 0 -> 2
- net /STM32F1/FMU_USART6_RX_IO_USART2_TX: track 0.00 -> 41.8 mm, vias 0 -> 2
- net /UART2_RX_TELEM3: track 0.00 -> 34.7 mm, vias 0 -> 2
- net /UART5_RX_TELEM2: track 0.00 -> 7.68 mm, vias 0 -> 2
- net GND: track 154.4 -> 152.4 mm, vias 314 -> 319
- net /UART5_TX_TELEM2: track 0.00 -> 1.58 mm, vias 0 -> 1
- net /UART7_TX_TELEM1: track 0.00 -> 1.53 mm, vias 0 -> 1
- net /UART7_RTS_TELEM1: track 0.00 -> 1.52 mm, vias 0 -> 1
- net /UART7_RX_TELEM1: track 0.00 -> 1.48 mm, vias 0 -> 1
- net /UART5_RTS_TELEM2: track 0.00 -> 1.43 mm, vias 0 -> 1
- net /UART5_CTS_TELEM2: track 0.00 -> 1.43 mm, vias 0 -> 1
- net /UART7_CTS_TELEM1: track 0.00 -> 1.38 mm, vias 0 -> 1

Commit message: Almost finish with initial routing
Parts:
- moved R97 35.7 mm to (113.2, 125.0), turned to 0 degrees
- moved C4 6.88 mm to (138.8, 98.5), turned to 180 degrees
- moved C53 5.96 mm to (107.0, 91.0), turned to 90 degrees
- moved C57 4.74 mm to (109.5, 95.5), turned to 0 degrees
- moved U56 4.15 mm to (111.4, 90.1), turned to -90 degrees
- moved R99 3.80 mm to (132.2, 104.3), turned to 180 degrees
- moved C3 2.27 mm to (135.8, 104.7)
- moved C59 1.91 mm to (109.5, 93.7), turned to 0 degrees
- moved X2 1.71 mm to (137.0, 102.0)
- moved R11 1.55 mm to (116.5, 87.5)
- moved C56 0.69 mm to (156.4, 114.2), turned to 180 degrees
- moved R98 0.14 mm to (118.2, 124.9)
Routing:
- net /UART5_RX_TELEM2: track 7.68 -> 154.0 mm
- net /UART7_RX_TELEM1: track 1.48 -> 91.9 mm, vias 1 -> 2
- net /UART5_RTS_TELEM2: track 1.43 -> 87.3 mm, vias 1 -> 2
- net /UART5_CTS_TELEM2: track 1.43 -> 82.0 mm, vias 1 -> 2
- net /UART5_TX_TELEM2: track 1.58 -> 75.1 mm, vias 1 -> 2
- net /SPI1_SCK: track 0.00 -> 65.9 mm, vias 0 -> 2
- net Net-(J15-Pad2): track 0.00 -> 63.4 mm, vias 0 -> 2
- net /SPI3_MOSI: track 0.00 -> 62.0 mm, vias 0 -> 2
- net /SPI3_MISO: track 0.00 -> 61.9 mm, vias 0 -> 2
- net /UART1_RX_GPS1: track 0.00 -> 61.7 mm, vias 0 -> 3
- net /UART8_RX_GPS2: track 0.00 -> 55.7 mm, vias 0 -> 4
- net /I2C1_SDA: track 0.00 -> 55.5 mm, vias 0 -> 2
- net /UART7_RTS_TELEM1: track 1.52 -> 57.0 mm, vias 1 -> 2
- net /SPI3_SCK: track 0.00 -> 54.0 mm, vias 0 -> 2
- net /I2C1_SCL: track 0.00 -> 53.0 mm, vias 0 -> 2
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