File: flight_controller/ETH.kicad_sch (KiCad schematic)
At the start: 29 parts, among them J15 HR911105A_C12074, U10 LAN8742AI-CZ, U8 LAN8742A, X4 X322525MOB4SI

Commit message: cleanup and improvements
Parts:
- removed U10: LAN8742AI-CZ, easyeda2kicad:QFN-24_L4.0-W4.0-P0.50-BL-EP2.6, symbol lampelKicadLIB:LAN8742AI-CZ
- removed U8: LAN8742A, Package_DFN_QFN:VQFN-24-1EP_4x4mm_P0.5mm_EP2.5x2.5mm_ThermalVias, symbol Interface_Ethernet:LAN8742A
- added U3: LAN8742AI-CZ, easyeda2kicad:QFN-24_L4.0-W4.0-P0.50-BL-EP2.6, symbol lampelKicadLIB:LAN8742AI-CZ
Connections:
- net 3V3: now also U3.1 (VDD2A), U3.19 (VDD1A), U3.9 (VDDIO)
- net ETH_LED1: now also U3.3 (LED1/REGOFF)
- net ETH_LED2: now also U3.2 (LED2/~{INTSEL})
- net ETH_MDC: now also U3.13 (MDC)
- net ETH_MDIO: now also U3.12 (MDIO)
- net ETH_NRST: now also U3.15 (~{RST})
- net ETH_RXN: now also U3.22 (RXN)
- net ETH_RXP: now also U3.23 (RXP)
- net ETH_TXD0: now also U3.17 (TXD0)
- net ETH_TXD1: now also U3.18 (TXD1)
- net ETH_TXN: now also U3.20 (TXN)
- net ETH_TXP: now also U3.21 (TXP)
- net ETH_TX_EN: now also U3.16 (TXEN)
- net GND: now also U3.25 (VSS)
- net at C63.2, C66.2: now also U3.6 (VDDCR)
- net at R75.2: now also U3.14 (~{INT}/REFCLKO)
- net at R93.1: now also U3.10 (RXER/PHYAD0)
- net at R76.2: now also U3.8 (RXD0/MODE0)
- net at R20.1: now also U3.24 (RBIAS)
- net at R29.2: now also U3.11 (CRS_DV/MODE2)
- net at C60.2, X4.1 (OSC1): now also U3.5 (XTAL1/CLKIN)
- net at C59.2, X4.3 (OSC2): now also U3.4 (XTAL2)
- net at R77.2: now also U3.7 (RXD1/MODE1)
Changed lines of the file:
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@@
-	)
-	(symbol
-		(lib_id "lampelKicadLIB:LAN8742AI-CZ")
-		(at 356.87 57.15 0)
-		(unit 1)
-		(exclude_from_sim no)
-		(in_bom yes)
-		(on_board yes)
-		(dnp no)
-		(fields_autoplaced yes)
-		(property "Reference" "U10"
-			(at 356.87 34.29 0)
-			(effects
-				(font
-					(size 1.27 1.27)
-				)
-			)
-		)
-		(property "Value" "LAN8742AI-CZ"
-			(at 356.87 36.83 0)
-			(effects
-				(font
-					(size 1.27 1.27)
-				)
-			)
-		)
-		(property "Footprint" "easyeda2kicad:QFN-24_L4.0-W4.0-P0.50-BL-EP2.6"
-			(at 356.87 80.01 0)
-			(effects
-				(font
-					(size 1.27 1.27)
-				)
-				(hide yes)
-			)
-		)
-		(property "Datasheet" "https://www.lcsc.com/product-detail/C153279.html"
-			(at 356.87 67.31 0)
-			(effects
-				(font
-					(size 1.27 1.27)
-				)
-				(hide yes)
-			)
-		)
-		(property "Description" "1.8V~3.3V PHY Transceiver RMII QFN-24-EP(4x4) Drivers, Receivers, Transceivers RoHS"
-			(at 356.87 57.15 0)
-			(effects
-				(font
-					(size 1.27 1.27)
-				)
-				(hide yes)
-			)
-		)
-		(property "LCSC Part" "C153279"
-			(at 356.87 85.09 0)
-			(effects
-				(font
-					(size 1.27 1.27)
-				)
-				(hide yes)
-			)
-		)
-		(pin "17"
-		)
-		(pin "6"
-		)
-		(pin "3"
-		)
-		(pin "24"
-		)
-		(pin "25"
-		)
-		(pin "23"
-		)
-		(pin "7"
-		)
-		(pin "1"
-		)
-		(pin "9"
-		)
-		(pin "5"
-		)
-		(pin "8"
-		)
-		(pin "11"
-		)
-		(pin "10"
-		)
-		(pin "19"
-		)
-		(pin "18"
-		)
-		(pin "21"
-		)
-		(pin "15"
-		)
-		(pin "13"
-		)
-		(pin "4"
-		)
-		(pin "14"
-		)
-		(pin "16"
-		)
-		(pin "20"
-		)
-		(pin "2"
-		)
-		(pin "12"
-		)
-		(pin "22"
-		)
-		(instances
-			(project "FP_BOARD"
-				(path "/17737359-1a8e-4237-8899-d9604030bc1d/050f1722-2ce7-4fbb-bd7f-6402b811e163"
-					(reference "U10")
-					(unit 1)
-				)
-			)
-		)
 	)
 	(symbol
@@
 	)
 	(symbol
-		(lib_id "Interface_Ethernet:LAN8742A")
-		(at 118.11 90.17 0)
-		(unit 1)
-		(exclude_from_sim no)
-		(in_bom yes)
-		(on_board yes)
-		(dnp no)
-		(fields_autoplaced yes)
-		(property "Reference" "U8"
-			(at 120.2533 118.11 0)
-			(effects
-				(font
-					(size 1.27 1.27)
-				)
-				(justify left)
-			)
-		)
-		(property "Value" "LAN8742A"
-			(at 120.2533 120.65 0)
-			(effects
-				(font
-					(size 1.27 1.27)
-				)
-				(justify left)
-			)
-		)
-		(property "Footprint" "Package_DFN_QFN:VQFN-24-1EP_4x4mm_P0.5mm_EP2.5x2.5mm_ThermalVias"
-			(at 119.38 116.84 0)
-			(effects
-				(font
-					(size 1.27 1.27)
-				)
-				(justify left)
-				(hide yes)
-			)
-		)
-		(property "Datasheet" "http://ww1.microchip.com/downloads/en/DeviceDoc/8742a.pdf"
-			(at 118.11 129.54 0)
-			(effects
-				(font
-					(size 1.27 1.27)
-				)
-				(hide yes)
-			)
-		)
-		(property "Description" "LAN8720 Ethernet PHY with RMII interface, QFN-24"
-			(at 118.11 90.17 0)
-			(effects
-				(font
-					(size 1.27 1.27)
-				)
-				(hide yes)
-			)
-		)
-		(pin "17"
-		)
-		(pin "11"
-		)
-		(pin "5"
-		)
-		(pin "9"
-		)
-		(pin "8"
-		)
-		(pin "6"
-		)
-		(pin "23"
-		)
-		(pin "13"
-		)
-		(pin "24"
-		)
-		(pin "15"
-		)
-		(pin "3"
-		)
-		(pin "1"
-		)
-		(pin "4"
-		)
-		(pin "25"
-		)
-		(pin "14"
-		)
-		(pin "7"
-		)
-		(pin "19"
-		)
-		(pin "12"
-		)
-		(pin "22"
-		)
-		(pin "10"
-		)
-		(pin "16"
-		)
-		(pin "21"
-		)
-		(pin "20"
-		)
-		(pin "18"
-		)
-		(pin "2"
-		)
-		(instances
-			(project ""
-				(path "/17737359-1a8e-4237-8899-d9604030bc1d/050f1722-2ce7-4fbb-bd7f-6402b811e163"
-					(reference "U8")
-					(unit 1)
-				)
-			)
-		)
-	)
-	(symbol
 		(lib_id "power:GND")
 		(at 205.74 59.69 0)
@@
 					(unit 1)
 				)
+			)
+		)
+	)
+	(symbol
+		(lib_id "lampelKicadLIB:LAN8742AI-CZ")
+		(at 118.11 90.17 0)
+		(unit 1)
+		(exclude_from_sim no)
+		(in_bom yes)
+		(on_board yes)
+		(dnp no)
+		(fields_autoplaced yes)
+		(property "Reference" "U3"
+			(at 123.952 117.602 0)
+			(do_not_autoplace yes)
+			(effects
+				(font
+					(size 1.27 1.27)
+				)
+			)
+		)
+		(property "Value" "LAN8742AI-CZ"
+			(at 130.048 120.396 0)
+			(do_not_autoplace yes)
+			(effects
+				(font
+					(size 1.27 1.27)
+				)
+			)
+		)
+		(property "Footprint" "easyeda2kicad:QFN-24_L4.0-W4.0-P0.50-BL-EP2.6"
+			(at 117.856 138.176 0)
+			(effects
+				(font
+					(size 1.27 1.27)
+				)
+				(hide yes)
+			)
+		)
+		(property "Datasheet" "https://www.lcsc.com/product-detail/C153279.html"
+			(at 118.364 146.558 0)
+			(effects
+				(font
+					(size 1.27 1.27)
+				)
+				(hide yes)
+			)
+		)
+		(property "Description" "1.8V~3.3V PHY Transceiver RMII QFN-24-EP(4x4) Drivers, Receivers, Transceivers RoHS"
+			(at 118.11 141.732 0)
+			(effects
+				(font
+					(size 1.27 1.27)
+				)
+				(hide yes)
+			)
+		)
+		(property "LCSC Part" "C153279"
+			(at 117.856 133.604 0)
+			(effects
+				(font
+					(size 1.27 1.27)
+				)
+				(hide yes)
+			)
+		)
+		(pin "18"
+		)
+		(pin "9"
+		)
+		(pin "5"
+		)
+		(pin "25"
+		)
+		(pin "15"
+		)
+		(pin "24"
+		)
+		(pin "12"
+		)
+		(pin "6"
+		)
+		(pin "16"
+		)
+		(pin "7"
+		)
+		(pin "21"
+		)
+		(pin "20"
+		)
+		(pin "23"
+		)
+		(pin "1"
+		)
+		(pin "4"
+		)
+		(pin "11"
+		)
+		(pin "13"
+		)
+		(pin "22"
+		)
+		(pin "3"
+		)
+		(pin "2"
+		)
+		(pin "17"
+		)
+		(pin "8"
+		)
+		(pin "10"
+		)
+		(pin "14"
+		)
+		(pin "19"
+		)
+		(instances
+			(project ""
+				(path "/17737359-1a8e-4237-8899-d9604030bc1d/050f1722-2ce7-4fbb-bd7f-6402b811e163"
+					(reference "U3")
+					(unit 1)
+				)

Commit message: Schematic complete, ready for layout. Added USB, TPs, power conn, updated clocks, ran Rules Checker and general review
Parts:
- removed C59, C60: CL10C120JB8NNNC ( 12pf , 0603 , 50v , C0G), easyeda2kicad:C0603, symbol lampelKicadLIB:CL10C120JB8NNNC ( 12pf , 0603 , 50v , C0G)
- removed X4: X322525MOB4SI, easyeda2kicad:CRYSTAL-SMD_4P-L3.2-W2.5-BL, symbol lampelKicadLIB:X322525MOB4SI
- added C52, C59: CC0603JRNPO9BN100 (10pF , 0603 ,50V ,X7R), easyeda2kicad:C0603, symbol lampelKicadLIB:CC0603JRNPO9BN100 (10pF , 0603 ,50V ,X7R)
- added X4: XL2EL89CMI-111YLC-25M, easyeda2kicad:CRYSTAL-SMD_4P-L3.2-W2.5-BL_SIT8008BI, symbol lampelKicadLIB:XL2EL89CMI-111YLC-25M
Connections:
- net GND: now also C52.1, C59.1, X4.2 (GND), X4.4 (GND)
- net at U3.5 (XTAL1/CLKIN): now also C59.2, X4.1
- net at U3.4 (XTAL2): now also C52.2, X4.3
Other:
- note added: "Crystal 25MHz"
Changed lines of the file:
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@@
 		)
 	)
+	(text "Crystal\n25MHz"
+		(exclude_from_sim no)
+		(at 54.356 122.174 0)
+		(effects
+			(font
+				(size 1.27 1.27)
+			)
+		)
+	)
 	(text "LEDS are\nActive high mode "
 		(exclude_from_sim no)
@@
 	)
 	(symbol
-		(lib_id "lampelKicadLIB:CL10C120JB8NNNC ( 12pf , 0603 , 50v , C0G)")
+		(lib_id "lampelKicadLIB:CC0603JRNPO9BN100 (10pF , 0603 ,50V ,X7R)")
 		(at 72.39 116.84 0)
 		(unit 1)
@@
 		(dnp no)
 		(fields_autoplaced yes)
-		(property "Reference" "C60"
+		(property "Reference" "C59"
 			(at 72.39 113.792 0)
 			(do_not_autoplace yes)
@@
 			)
 		)
-		(property "Value" "CL10C120JB8NNNC ( 12pf , 0603 , 50v , C0G)"
+		(property "Value" "CC0603JRNPO9BN100 (10pF , 0603 ,50V ,X7R)"
 			(at 72.39 121.92 0)
 			(effects
@@
 			)
 		)
-		(property "Datasheet" "https://lcsc.com/product-detail/Multilayer-Ceramic-Capacitors-MLCC-SMD-SMT_SAMSUNG_CL10C120JB8NNNC_12pF-120-5-50V_C38523.html"
+		(property "Datasheet" "https://www.lcsc.com/product-detail/C106245.html"
 			(at 72.39 127 0)
 			(effects
@@
 			)
 		)
-		(property "Description" "12pF ±5% 50V Ceramic Capacitor C0G 0603"
-			(at 72.39 116.84 0)
+		(property "Description" "10pF ±5% 50V Ceramic Capacitor NP0 0603"
+			(at 72.39 132.08 0)
 			(effects
 				(font
@@
 			)
 		)
-		(property "LCSC Part" "C38523"
+		(property "LCSC Part" "C106245"
 			(at 72.39 129.54 0)
 			(effects
@@
 			(project "FP_BOARD"
 				(path "/17737359-1a8e-4237-8899-d9604030bc1d/050f1722-2ce7-4fbb-bd7f-6402b811e163"
-					(reference "C60")
-					(unit 1)
-				)
-			)
-		)
-	)
-	(symbol
-		(lib_id "lampelKicadLIB:CL10C120JB8NNNC ( 12pf , 0603 , 50v , C0G)")
-		(at 33.02 116.84 0)
-		(unit 1)
-		(exclude_from_sim no)
-		(in_bom yes)
-		(on_board yes)
-		(dnp no)
-		(fields_autoplaced yes)
-		(property "Reference" "C59"
-			(at 33.02 113.792 0)
-			(do_not_autoplace yes)
-			(effects
-				(font
-					(size 1.27 1.27)
-				)
-			)
-		)
-		(property "Value" "CL10C120JB8NNNC ( 12pf , 0603 , 50v , C0G)"
-			(at 33.02 121.92 0)
-			(effects
-				(font
-					(size 1.27 1.27)
-				)
-				(hide yes)
-			)
-		)
-		(property "Footprint" "easyeda2kicad:C0603"
-			(at 33.02 124.46 0)
-			(effects
-				(font
-					(size 1.27 1.27)
-				)
-				(hide yes)
-			)
-		)
-		(property "Datasheet" "https://lcsc.com/product-detail/Multilayer-Ceramic-Capacitors-MLCC-SMD-SMT_SAMSUNG_CL10C120JB8NNNC_12pF-120-5-50V_C38523.html"
-			(at 33.02 127 0)
-			(effects
-				(font
-					(size 1.27 1.27)
-				)
-				(hide yes)
-			)
-		)
-		(property "Description" "12pF ±5% 50V Ceramic Capacitor C0G 0603"
-			(at 33.02 116.84 0)
-			(effects
-				(font
-					(size 1.27 1.27)
-				)
-				(hide yes)
-			)
-		)
-		(property "LCSC Part" "C38523"
-			(at 33.02 129.54 0)
-			(effects
-				(font
-					(size 1.27 1.27)
-				)
-				(hide yes)
-			)
-		)
-		(pin "1"
-		)
-		(pin "2"
-		)
-		(instances
-			(project "FP_BOARD"
-				(path "/17737359-1a8e-4237-8899-d9604030bc1d/050f1722-2ce7-4fbb-bd7f-6402b811e163"
 					(reference "C59")
 					(unit 1)
@@
 	)
 	(symbol
+		(lib_id "lampelKicadLIB:XL2EL89CMI-111YLC-25M")
+		(at 54.61 114.3 180)
+		(unit 1)
+		(exclude_from_sim no)
+		(in_bom yes)
+		(on_board yes)
+		(dnp no)
+		(property "Reference" "X4"
+			(at 54.61 106.172 0)
+			(effects
+				(font
+					(size 1.27 1.27)
+				)
+			)
+		)
+		(property "Value" "XL2EL89CMI-111YLC-25M"
+			(at 54.61 108.204 0)
+			(effects
+				(font
+					(size 1.27 1.27)
+				)
+			)
+		)
+		(property "Footprint" "easyeda2kicad:CRYSTAL-SMD_4P-L3.2-W2.5-BL_SIT8008BI"
+			(at 54.61 104.14 0)
+			(effects
+				(font
+					(size 1.27 1.27)
+				)
+				(hide yes)
+			)
+		)
+		(property "Datasheet" "https://www.lcsc.com/product-detail/C5444611.html"
+			(at 54.61 104.14 0)
+			(effects
+				(font
+					(size 1.27 1.27)
+				)
+				(hide yes)
+			)
+		)
+		(property "Description" "Crystal 25MHz ±10ppm 10pF SMD3225-4P"
+			(at 54.61 114.3 0)
+			(effects
+				(font
+					(size 1.27 1.27)
+				)
+				(hide yes)
+			)
+		)
+		(property "LCSC Part" "C5444611"
+			(at 54.61 101.6 0)
+			(effects
+				(font
+					(size 1.27 1.27)
+				)
+				(hide yes)
+			)
+		)
+		(pin "2"
+		)
+		(pin "4"
+		)
+		(pin "1"
+		)
+		(pin "3"
+		)
+		(instances
+			(project ""
+				(path "/17737359-1a8e-4237-8899-d9604030bc1d/050f1722-2ce7-4fbb-bd7f-6402b811e163"
+					(reference "X4")
+					(unit 1)
+				)
+			)
+		)
+	)
+	(symbol
 		(lib_id "easyeda2kicad:0603WAF1002T5E")
 		(at 167.64 110.49 270)
@@
 	)
 	(symbol
-		(lib_id "lampelKicadLIB:X322525MOB4SI")
-		(at 54.61 114.3 0)
+		(lib_id "lampelKicadLIB:CC0603JRNPO9BN100 (10pF , 0603 ,50V ,X7R)")
+		(at 33.02 116.84 0)
 		(unit 1)
 		(exclude_from_sim no)
@@
 		(dnp no)
 		(fields_autoplaced yes)
-		(property "Reference" "X4"
-			(at 54.61 106.172 0)
+		(property "Reference" "C52"
+			(at 33.02 113.792 0)
 			(do_not_autoplace yes)
 			(effects
@@
 			)
 		)
-		(property "Value" "X322525MOB4SI"
-			(at 55.372 108.204 0)
-			(do_not_autoplace yes)
+		(property "Value" "CC0603JRNPO9BN100 (10pF , 0603 ,50V ,X7R)"
+			(at 33.02 121.92 0)
 			(effects
 				(font
 					(size 1.27 1.27)
 				)
+				(hide yes)
 			)
 		)
-		(property "Footprint" "easyeda2kicad:CRYSTAL-SMD_4P-L3.2-W2.5-BL"
-			(at 54.61 124.46 0)
+		(property "Footprint" "easyeda2kicad:C0603"
+			(at 33.02 124.46 0)
 			(effects
 				(font
@@
 			)
 		)
-		(property "Datasheet" "https://lcsc.com/product-detail/SMD-Crystals_YSX321SL-25MHZ-12PF-10PPM-40-85_C9006.html"
-			(at 54.61 127 0)
+		(property "Datasheet" "https://www.lcsc.com/product-detail/C106245.html"
+			(at 33.02 127 0)
 			(effects
 				(font
@@
 			)
 		)
-		(property "Description" "Crystal 25MHz ±10ppm 12pF SMD3225-4P"
-			(at 54.61 133.858 0)
+		(property "Description" "10pF ±5% 50V Ceramic Capacitor NP0 0603"
+			(at 33.02 132.08 0)
 			(effects
 				(font
@@
 			)
 		)
-		(property "LCSC Part" "C9006"
-			(at 54.61 129.54 0)
+		(property "LCSC Part" "C106245"
+			(at 33.02 129.54 0)
 			(effects
 				(font
@@
 			)
 		)
-		(pin "2"
-		)
-		(pin "4"
-		)
 		(pin "1"
 		)
-		(pin "3"
+		(pin "2"
 		)
 		(instances
 			(project "FP_BOARD"
 				(path "/17737359-1a8e-4237-8899-d9604030bc1d/050f1722-2ce7-4fbb-bd7f-6402b811e163"
-					(reference "X4")
+					(reference "C52")
 					(unit 1)
 				)

Commit message: Started the placement process
Parts:
- renumbered C52 to C63, C59 to C64, C63 to C65, C62 to C66, C66 to C67, C65 to C68, C7 to C69, C8 to C70, C64 to C71, C61 to C72, J15 to J14, R81 to R71, R21 to R72, R93 to R73, R76 to R74, R77 to R75, R29 to R76, R75 to R77, R82 to R78, R20 to R79, R87 to R80, R90 to R81, R88 to R82, R89 to R83, R92 to R84, R91 to R85, U3 to U14

Commit message: Updated power and usb connectors, annotations and netlist check
Parts:
- renumbered J14 to J16, R71 to R70, R72 to R71, R73 to R72, R74 to R73, R75 to R74, R76 to R75, R77 to R76, R78 to R77, R79 to R78, R80 to R79, R81 to R80, R82 to R81, R83 to R82, R84 to R83, R85 to R84, U14 to U12

Commit message: Revert to state of commit 2458262 moved all to components to top
Reverts commits: d012532, 3d9c600, 58bc0ac
Parts:
- renumbered J16 to J14, R70 to R71, R71 to R72, R72 to R73, R73 to R74, R74 to R75, R75 to R76, R76 to R77, R77 to R78, R78 to R79, R79 to R80, R80 to R81, R81 to R82, R82 to R83, R83 to R84, R84 to R85, U12 to U14

Commit message: Changed eth net name and started diff route , added custom rules file for diff
Connections:
- net ETH_RXN renamed ETH_RX_N
- net ETH_RXP renamed ETH_RX_P
- net ETH_TXN renamed ETH_TX_N
- net ETH_TXP renamed ETH_TX_P
Changed lines of the file:
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@@
 		)
 	)
-	(label "ETH_TXN"
+	(label "ETH_TX_N"
 		(at 198.12 80.01 0)
 		(effects
@@
 		)
 	)
-	(label "ETH_RXN"
+	(label "ETH_RX_N"
 		(at 139.7 85.09 0)
 		(effects
@@
 		)
 	)
-	(label "ETH_TXP"
+	(label "ETH_TX_P"
 		(at 139.7 77.47 0)
 		(effects
@@
 		)
 	)
-	(label "ETH_RXP"
+	(label "ETH_RX_P"
 		(at 198.12 74.93 0)
 		(effects
@@
 		)
 	)
-	(label "ETH_RXP"
+	(label "ETH_RX_P"
 		(at 139.7 82.55 0)
 		(effects
@@
 		)
 	)
-	(label "ETH_TXP"
+	(label "ETH_TX_P"
 		(at 198.12 85.09 0)
 		(effects
@@
 		)
 	)
-	(label "ETH_RXN"
+	(label "ETH_RX_N"
 		(at 198.12 69.85 0)
 		(effects
@@
 		)
 	)
-	(label "ETH_TXN"
+	(label "ETH_TX_N"
 		(at 139.7 80.01 0)
 		(effects

Commit message: Added stuff
Parts:
- removed C68: CL10B103KB8NNNC (10nf , 0603 , 50v , X7R), easyeda2kicad:C0603, symbol lampelKicadLIB:CL10B103KB8NNNC (10nf , 0603 , 50v , X7R)
- removed C71: CL10A106MA8NRNC (10uf , 0603 ,25v ,X5R), easyeda2kicad:C0603, symbol lampelKicadLIB:CL10A106MA8NRNC (10uf , 0603 ,25v ,X5R)
