File: flight_controller/SERVO_RC.kicad_sch (KiCad schematic)
At the start: 30 parts, among them J10 HX PZ2.54-3X4P ZZ, J13 HX PZ2.54-3X4P ZZ, J14 B3B-ZR-SM4-TF(LF)(SN), J3 HX PZ2.54-3X4P ZZ, J4 HX PZ2.54-3X4P ZZ, J9 HX PZ2.54-3X4P ZZ, U11 STM32H753IIT6, U7 SN74LVC2G240DCTR

Commit message: cleanup and improvements
Parts:
- removed J3, J9: HX PZ2.54-3X4P ZZ, easyeda2kicad:HDR-TH_12P-P2.54-V-M-R3-C4-S2.54, symbol lampelKicadLIB:HXPZ2.54-3X4PZZ
- removed R26, R27, R28, R6, R7: 0603WAF2200T5E (220ohm , 0603), easyeda2kicad:R0603, symbol lampelKicadLIB:0603WAF2200T5E (220ohm , 0603)
- added C68: CC0603KRX7R9BB104 (100nf , 0603 ,50v ,X7R), easyeda2kicad:C0603, symbol lampelKicadLIB:CC0603KRX7R9BB104 (100nf , 0603 ,50v ,X7R)
Connections:
- net 3V3: now also C68.2
- net GND: now also C68.1

Commit message: Schematic complete, ready for layout. Added USB, TPs, power conn, updated clocks, ran Rules Checker and general review
Other:
- note added: "Spare FMU_CH"
- note added: "Spare IO_CH"
- note added: "Use FMU_CH as PWM or DShot for Motors"
- note added: "Use IO_CH as PWM for Servo"
- note removed: "SERVO"
- note removed: "SERVO FMC"
- note removed: "SERVO IO"
Changed lines of the file:
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@@
 	(generator_version "9.0")
 	(paper "A2")
-	(text "SERVO\nIO"
+	(text "Use IO_CH\nas PWM\nfor Servo"
 		(exclude_from_sim no)
-		(at 418.084 222.504 0)
+		(at 419.354 223.012 0)
 		(effects
 			(font
@@
 		)
 	)
-	(text "SERVO"
+	(text "Spare FMU_CH"
 		(exclude_from_sim no)
-		(at 421.64 79.248 0)
+		(at 423.418 75.438 0)
 		(effects
 			(font
@@
 		)
 	)
-	(text "SERVO\nFMC"
+	(text "Use FMU_CH as\nPWM or DShot\nfor Motors"
 		(exclude_from_sim no)
-		(at 420.37 147.574 0)
+		(at 427.228 149.86 0)
 		(effects
 			(font
@@
 		(effects
 			(font
+				(size 2.54 2.54)
+			)
+		)
+	)
+	(text "Spare IO_CH"
+		(exclude_from_sim no)
+		(at 421.386 83.058 0)
+		(effects
+			(font

Commit message: Started the placement process
Parts:
- removed U11: STM32H753IIT6, easyeda2kicad:LQFP-176_L24.0-W24.0-P0.50-BL, symbol easyeda2kicad:STM32H753IIT6
- renumbered C57 to C37, C68 to C38, J10 to J1, J14 to J2, J4 to J3, J13 to J4, R80 to R26, R85 to R27, R84 to R28, R79 to R29, R83 to R30, R30 to R31, R31 to R32, R32 to R33, R33 to R34, R22 to R35, R23 to R36, R24 to R37, R25 to R38, R72 to R39, R74 to R40, R78 to R41, U7 to U5

Commit message: Updated power and usb connectors, annotations and netlist check
Parts:
- renumbered J1 to J3, J2 to J4, J3 to J5, J4 to J6, U5 to U3
Changed lines of the file:
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@@
 		(dnp no)
 		(fields_autoplaced yes)
-		(property "Reference" "J3"
+		(property "Reference" "J5"
 			(at 398.78 131.064 0)
 			(do_not_autoplace yes)
@@
 			(project "FP_BOARD"
 				(path "/17737359-1a8e-4237-8899-d9604030bc1d/a3423b8d-b0bd-4c78-958f-6f0b6cb1ee40"
-					(reference "J3")
+					(reference "J5")
 					(unit 1)
 				)
@@
 		(dnp no)
 		(fields_autoplaced yes)
-		(property "Reference" "J4"
+		(property "Reference" "J6"
 			(at 401.32 56.134 0)
 			(do_not_autoplace yes)
@@
 			(project "FP_BOARD"
 				(path "/17737359-1a8e-4237-8899-d9604030bc1d/a3423b8d-b0bd-4c78-958f-6f0b6cb1ee40"
-					(reference "J4")
+					(reference "J6")
 					(unit 1)
 				)
@@
 		(dnp no)
 		(fields_autoplaced yes)
-		(property "Reference" "J2"
+		(property "Reference" "J4"
 			(at 406.4 310.642 0)
 			(do_not_autoplace yes)
@@
 			(project ""
 				(path "/17737359-1a8e-4237-8899-d9604030bc1d/a3423b8d-b0bd-4c78-958f-6f0b6cb1ee40"
-					(reference "J2")
+					(reference "J4")
 					(unit 1)
 				)
@@
 		(dnp no)
 		(fields_autoplaced yes)
-		(property "Reference" "J1"
+		(property "Reference" "J3"
 			(at 394.97 205.994 0)
 			(do_not_autoplace yes)
@@
 			(project "FP_BOARD"
 				(path "/17737359-1a8e-4237-8899-d9604030bc1d/a3423b8d-b0bd-4c78-958f-6f0b6cb1ee40"
-					(reference "J1")
+					(reference "J3")
 					(unit 1)
 				)
@@
 		(on_board yes)
 		(dnp no)
-		(property "Reference" "U5"
+		(property "Reference" "U3"
 			(at 227.33 54.61 0)
 			(effects
@@
 			(project ""
 				(path "/17737359-1a8e-4237-8899-d9604030bc1d/a3423b8d-b0bd-4c78-958f-6f0b6cb1ee40"
-					(reference "U5")
-					(unit 1)
-				)
+					(reference "U3")
+					(unit 1)
+				)

Commit message: Revert to state of commit 2458262 moved all to components to top
Reverts commits: d012532, 3d9c600, 58bc0ac
Parts:
- renumbered J3 to J1, J4 to J2, J5 to J3, J6 to J4, U3 to U5
Changed lines of the file:
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@@
 		(dnp no)
 		(fields_autoplaced yes)
-		(property "Reference" "J5"
+		(property "Reference" "J3"
 			(at 398.78 131.064 0)
 			(do_not_autoplace yes)
@@
 			(project "FP_BOARD"
 				(path "/17737359-1a8e-4237-8899-d9604030bc1d/a3423b8d-b0bd-4c78-958f-6f0b6cb1ee40"
-					(reference "J5")
+					(reference "J3")
 					(unit 1)
 				)
@@
 		(dnp no)
 		(fields_autoplaced yes)
-		(property "Reference" "J6"
+		(property "Reference" "J4"
 			(at 401.32 56.134 0)
 			(do_not_autoplace yes)
@@
 			(project "FP_BOARD"
 				(path "/17737359-1a8e-4237-8899-d9604030bc1d/a3423b8d-b0bd-4c78-958f-6f0b6cb1ee40"
-					(reference "J6")
+					(reference "J4")
 					(unit 1)
 				)
@@
 		(dnp no)
 		(fields_autoplaced yes)
-		(property "Reference" "J4"
+		(property "Reference" "J2"
 			(at 406.4 310.642 0)
 			(do_not_autoplace yes)
@@
 			(project ""
 				(path "/17737359-1a8e-4237-8899-d9604030bc1d/a3423b8d-b0bd-4c78-958f-6f0b6cb1ee40"
-					(reference "J4")
+					(reference "J2")
 					(unit 1)
 				)
@@
 		(dnp no)
 		(fields_autoplaced yes)
-		(property "Reference" "J3"
+		(property "Reference" "J1"
 			(at 394.97 205.994 0)
 			(do_not_autoplace yes)
@@
 			(project "FP_BOARD"
 				(path "/17737359-1a8e-4237-8899-d9604030bc1d/a3423b8d-b0bd-4c78-958f-6f0b6cb1ee40"
-					(reference "J3")
+					(reference "J1")
 					(unit 1)
 				)
@@
 		(on_board yes)
 		(dnp no)
-		(property "Reference" "U3"
+		(property "Reference" "U5"
 			(at 227.33 54.61 0)
 			(effects
@@
 			(project ""
 				(path "/17737359-1a8e-4237-8899-d9604030bc1d/a3423b8d-b0bd-4c78-958f-6f0b6cb1ee40"
-					(reference "U3")
-					(unit 1)
-				)
+					(reference "U5")
+					(unit 1)
+				)

Commit message: Advanced in routing
Other:
- moved on the sheet: C38
Changed lines of the file:
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@@
 	(symbol
 		(lib_id "lampelKicadLIB:CC0603KRX7R9BB104 (100nf , 0603 ,50v ,X7R)")
-		(at 381 299.72 90)
+		(at 381 299.72 270)
+		(mirror x)
 		(unit 1)
 		(exclude_from_sim no)
@@
 		(on_board yes)
 		(dnp no)
-		(fields_autoplaced yes)
 		(property "Reference" "C38"
-			(at 378.206 299.72 0)
+			(at 383.794 299.72 0)
 			(do_not_autoplace yes)
 			(effects
@@
 		)
 		(property "Value" "CC0603KRX7R9BB104 (100nf , 0603 ,50v ,X7R)"
-			(at 386.08 299.72 0)
+			(at 375.92 299.72 0)
 			(effects
 				(font
@@
 		)
 		(property "Footprint" "easyeda2kicad:C0603"
-			(at 388.62 299.72 0)
+			(at 373.38 299.72 0)
 			(effects
 				(font
@@
 		)
 		(property "Datasheet" "https://lcsc.com/product-detail/Multilayer-Ceramic-Capacitors-MLCC-SMD-SMT_100nF-104-10-50V_C14663.html"
-			(at 391.16 299.72 0)
+			(at 370.84 299.72 0)
 			(effects
 				(font
@@
 		)
 		(property "LCSC Part" "C14663"
-			(at 393.7 299.72 0)
+			(at 368.3 299.72 0)
 			(effects
 				(font

Commit message: Finished Board and silkscreen
Parts:
- added R56: 603WAF0000T5E (0ohm , 0603), easyeda2kicad:R0603, symbol lampelKicadLIB:0603WAF0000T5E (0ohm , 0603)
Connections:
- net IO_USART1_RX_DSM: now also R56.2; no longer R41.1
- new net: R41.1, R56.1
Changed lines of the file:
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@@
 	(wire
 		(pts
-			(xy 364.49 314.96) (xy 344.17 314.96)
+			(xy 364.49 314.96) (xy 360.68 314.96)
 		)
 		(stroke
@@
 		(pts
 			(xy 358.14 82.55) (xy 391.16 82.55)
+		)
+		(stroke
+			(width 0)
+			(type default)
+		)
+	)
+	(wire
+		(pts
+			(xy 350.52 314.96) (xy 344.17 314.96)
 		)
 		(stroke
@@
 					(unit 1)
 				)
+			)
+		)
+	)
+	(symbol
+		(lib_id "lampelKicadLIB:0603WAF0000T5E (0ohm , 0603)")
+		(at 355.6 314.96 180)
+		(unit 1)
+		(exclude_from_sim yes)
+		(in_bom no)
+		(on_board yes)
+		(dnp yes)
+		(fields_autoplaced yes)
+		(property "Reference" "R56"
+			(at 355.6 316.992 0)
+			(do_not_autoplace yes)
+			(effects
+				(font
+					(size 1.27 1.27)
+				)
+			)
+		)
+		(property "Value" "603WAF0000T5E (0ohm , 0603)"
+			(at 355.6 309.88 0)
+			(effects
+				(font
+					(size 1.27 1.27)
+				)
+				(hide yes)
+			)
+		)
+		(property "Footprint" "easyeda2kicad:R0603"
+			(at 355.6 307.34 0)
+			(effects
+				(font
+					(size 1.27 1.27)
+				)
+				(hide yes)
+			)
+		)
+		(property "Datasheet" "https://lcsc.com/product-detail/Chip-Resistor-Surface-Mount-UniOhm_0R-0R0-1_C21189.html"
+			(at 355.6 304.8 0)
+			(effects
+				(font
+					(size 1.27 1.27)
+				)
+				(hide yes)
+			)
+		)
+		(property "Description" "0Ω ±1% 100mW 0603 Thick Film Resistor"
+			(at 355.6 299.72 0)
+			(effects
+				(font
+					(size 1.27 1.27)
+				)
+				(hide yes)
+			)
+		)
+		(property "LCSC Part" "C21189"
+			(at 355.6 302.26 0)
+			(effects
+				(font
+					(size 1.27 1.27)
+				)
+				(hide yes)
+			)
+		)
+		(pin "1"
+		)
+		(pin "2"
+		)
+		(instances
+			(project "FP_BOARD"
+				(path "/17737359-1a8e-4237-8899-d9604030bc1d/a3423b8d-b0bd-4c78-958f-6f0b6cb1ee40"
+					(reference "R56")
+					(unit 1)
+				)
